File: pcb/reeeflow-v3.sch (EAGLE design)
At the start: 64 parts, among them J1 SH-6, J2 DC-JACK, Q1 BC817-40, Q2 BC817-40, Q3 BC817-40, U1 EFM32GG11B8XX_Q100, U2 SST26VF064B, U3 MIC39100, U4 MCP9600, U5 ER-TFT035-6BOT, U7 MCP9600, Y1 32.768KHz, Y2 8MHz

Commit message: modified the sch slightly
Parts:
- removed U$5: HLK-PM01, Power > AC\DC Converters:HLK-PM01
- added B2, B3, B4, B5, B6: PUSH-SILENT, Eletromechanical > Switches > Tactile Switches:PUSH-SILENT
- added C19, C20, C21, C22, C23, C24: (no value), Passive Components > Capacitors > Multilayer Ceramic Capacitors MLCC:MLCC0603
- added R30, R31, R32, R33: (no value), Passive Components > Resistors > Chip Resistors:RESISTOR0603
- added SW1: (no value), Eletromechanical > Switches > Tactile Switches:PUSH_BUTTON
- J2: value DC-JACK -> PH-2; device Connectors > Jack:DC-JACK -> Connectors > JST > PH:PH-2
Connections:
- net !TFT_IRQ renamed !TFT-IRQ
- net I2C0_SCL_SENS renamed I2C0-SCL-SENS
- net I2C0_SDA_SENS renamed I2C0-SDA-SENS
- net I2C1_SCL_TFT renamed I2C1-SCL-TFT
- net I2C1_SDA_TFT renamed I2C1-SDA-TFT
- net N$33 renamed !TFT-RST
- net TFT_DC renamed TFT-DC
- net US1_CLK_TFT renamed US1-CLK-TFT
- net US1_CS_TFT renamed US1-CS-TFT
- net US1_MISO_TFT renamed US1-MISO-TFT
- net US1_MOSI_TFT renamed US1-MOSI-TFT
- removed net N$28: U$5.AC1
- removed net N$29: J2.2, J2.3, U$5.AC2
- removed net N$30: J2.1
- new net BTN_1: R30.P$2
- new net BTN_2: R15.P$2
- new net BTN_3: R31.P$2
- new net BTN_4: R32.P$2
- new net BTN_5: R33.P$2
- new net N$12: B5.3, C23.P$2, R13.P$1, R32.P$1
- new net N$14: B6.3, C24.P$2, R14.P$1, R33.P$1
- new net N$3: B2.3, C20.P$2, R10.P$1, R30.P$1
- new net N$6: B3.3, C21.P$2, R11.P$1, R15.P$1
- new net N$8: B4.3, C22.P$2, R12.P$1, R31.P$1
- new net TC0-ALRT1: U4.ALRT1@11
- new net TC0-ALRT2: U4.ALRT2@12
- new net TC0-ALRT3: U4.ALRT3@14
- new net TC0-ALRT4: U4.ALERT4@15
- new net TC1-ALRT1: U7.ALRT1@11
- new net TC1-ALRT2: U7.ALRT2@12
- new net TC1-ALRT3: U7.ALRT3@14
- new net TC1-ALRT4: U7.ALERT4@15
- net !RESET: now also SW1.1, SW1.2
- net 3.3V: now also C19.P$1, R10.P$2, R11.P$2, R12.P$2, R13.P$2, R14.P$2
- net GND: now also B2.1, B3.1, B4.1, B5.1, B6.1, C19.P$2, C20.P$1, C21.P$1, C22.P$1, C23.P$1, C24.P$1, J22.S, J2CASE.S, SW1.3, SW1.4; no longer U$5.-VO
- net N$31: now also J21.S; no longer U$5.+VO
Other:
- note added: "TODO: Buttons out coms interface (uart?)"
- note removed: "TODO: AC/DC adapter 3.3V regulator"
- note removed: "TODO: Display State Led Buzzer Buttons Encoder SD card reader? out coms interface (uart?)"
- note removed: "TODO: MCU CONNECTIONS"
- note removed: "fuse"
- note removed: "varistor"
- moved on the sheet: C13, C14, C6, F1, J11, J12, J13, J14, J15, J16, J1CASE, R10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

Commit message: modified the sch slightly
Parts:
- added C25: (no value), Passive Components > Capacitors > Multilayer Ceramic Capacitors MLCC:MLCC0603
Connections:
- net 3.3V: now also C25.P$1
- net GND: now also C25.P$2
Changed lines of the file:
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@@
 <part name="J2" library="Connectors &gt; JST &gt; PH" deviceset="PH-2" device=""/>
 <part name="GND39" library="Utility &gt; Power Symbols" deviceset="GND" device=""/>
+<part name="C25" library="Passive Components &gt; Capacitors &gt; Multilayer Ceramic Capacitors MLCC" deviceset="MLCC" device="0603"/>
+<part name="SUPPLY45" library="Utility &gt; Power Symbols" deviceset="3.3V" device=""/>
+<part name="GND40" library="Utility &gt; Power Symbols" deviceset="GND" device=""/>
 </parts>
 <sheets>
@@
 servo out's
 motor out's (door open)</text>
-<text x="16.256" y="229.616" size="1.778" layer="94" rot="R90">Decouple</text>
-<wire x1="20.32" y1="226.06" x2="1.27" y2="226.06" width="0.1016" layer="94"/>
-<wire x1="20.32" y1="226.06" x2="20.32" y2="251.46" width="0.1016" layer="94"/>
+<text x="23.876" y="229.616" size="1.778" layer="94" rot="R90">Decouple</text>
+<wire x1="27.94" y1="226.06" x2="1.27" y2="226.06" width="0.1016" layer="94"/>
+<wire x1="27.94" y1="226.06" x2="27.94" y2="251.46" width="0.1016" layer="94"/>
 </plain>
 <instances>
@@
 <instance part="SUPPLY36" gate="G$1" x="215.9" y="119.38" smashed="yes">
 <attribute name="VALUE" x="215.9" y="122.174" size="1.778" layer="96" align="bottom-center"/>
+</instance>
+<instance part="C25" gate="G$1" x="15.24" y="238.76" smashed="yes">
+<attribute name="NAME" x="13.716" y="236.22" size="1.27" layer="95" rot="R90"/>
+<attribute name="VALUE" x="17.78" y="236.22" size="1.27" layer="96" rot="R90"/>
+</instance>
+<instance part="SUPPLY45" gate="G$1" x="15.24" y="243.84" smashed="yes">
+<attribute name="VALUE" x="15.24" y="246.634" size="1.778" layer="96" align="bottom-center"/>
+</instance>
+<instance part="GND40" gate="1" x="15.24" y="231.14" smashed="yes">
+<attribute name="VALUE" x="15.24" y="230.886" size="1.778" layer="96" align="top-center"/>
 </instance>
 </instances>
@@
 <pinref part="U7" gate="G$1" pin="GND@18"/>
 </segment>
+<segment>
+<pinref part="C25" gate="G$1" pin="P$2"/>
+<pinref part="GND40" gate="1" pin="GND"/>
+<wire x1="15.24" y1="236.22" x2="15.24" y2="233.68" width="0.1524" layer="91"/>
+</segment>
 </net>
 <net name="3.3V" class="0">
@@
 <pinref part="SUPPLY36" gate="G$1" pin="3.3V"/>
 </segment>
-</net>
+<segment>
+<pinref part="SUPPLY45" gate="G$1" pin="3.3V"/>
+<pinref part="C25" gate="G$1" pin="P$1"/>
+<wire x1="15.24" y1="243.84" x2="15.24" y2="241.3" width="0.1524" layer="91"/>
+</segment>
+</net>
