File: pcb/reeeflow-v3.brd (EAGLE design)
At the start: 100 x 100 mm, 107 parts, among them J1 SH-6, J3 2EDG-2P, J4 2EDG-2P, J5 2EDG-2P, J6 2EDG-2P, J7 2EDG-2P, J8 3X1_2.54, J9 2X1_2.54, Q1 BC817-40, Q2 BC817-40, Q3 BC817-40, Q4 BC817-40, U1 EFM32GG11B8XX_Q64, U2 SST26VF064B, U3 MIC39100, U4 MCP9600, U5 ER-TFT035-6BOT, U6 H11AA1, U7 MCP9600, Y1 32.768KHz, Y2 8MHz

Commit message: pcb work
Parts:
- moved J1 201.7 mm to (96.6, 71.9), turned to 90 degrees
- moved D3 195.1 mm to (93.7, 28.4), turned to 90 degrees
- moved U$5 190.2 mm to (92.2, 20.7)
- moved SW1 189.9 mm to (95.6, 58.6), turned to 90 degrees
- moved D2 188.1 mm to (91.3, 28.6), turned to 270 degrees
- moved U4 172.7 mm to (79.0, 17.0), turned to 90 degrees
- moved U7 169.1 mm to (65.0, 17.0), turned to 90 degrees
- moved D4 160.0 mm to (92.4, 12.6)
- moved U2 149.1 mm to (50.0, 85.0)
- moved J8 141.8 mm to (54.0, 2.00)
- moved J9 132.9 mm to (46.0, 2.00)
- moved Y2 131.2 mm to (49.5, 59.7)
- moved Q4 127.3 mm to (92.4, 88.7), turned to 90 degrees
- moved R41 113.7 mm to (24.0, 14.0), turned to 90 degrees
- moved R40 109.6 mm to (20.0, 14.0), turned to 90 degrees
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Other:
- outline, holes or cut-outs redrawn
