File: pcb/r3eflow-v3.brd (EAGLE design)
At the start: 100 x 100 mm, 107 parts, among them J1 SH-6, J3 2EDG-2P, J4 2EDG-2P, J5 2EDG-2P, J6 2EDG-2P, J7 2EDG-2P, J8 3X1_2.54, J9 2X1_2.54, Q1 BC817-40, Q2 BC817-40, Q3 BC817-40, Q4 BC817-40, U1 EFM32GG11B8XX_Q64, U2 SST26VF064B, U3 MIC39100, U4 MCP9600, U5 ER-TFT035-6BOT, U6 H11AA1, U7 MCP9600, Y1 32.768KHz, Y2 8MHz

Commit message: updated gitignore
Parts:
- moved R6 133.3 mm to (-19.1, 3.24), turned to 90 degrees
- moved R32 132.0 mm to (-25.4, 4.51), turned to 90 degrees
- moved C12 130.8 mm to (-29.2, 5.78), turned to 90 degrees
- moved R5 127.9 mm to (-19.1, 7.05), turned to 90 degrees
- moved R31 126.6 mm to (-25.4, 8.32), turned to 90 degrees
- moved C11 123.6 mm to (-29.2, 10.9), turned to 90 degrees
- moved R4 122.5 mm to (-19.1, 10.9), turned to 90 degrees
- moved R30 121.2 mm to (-25.4, 12.1), turned to 90 degrees
- moved R3 117.2 mm to (-19.1, 14.7), turned to 90 degrees
- moved C10 116.5 mm to (-29.2, 15.9), turned to 90 degrees
- moved R29 115.9 mm to (-25.4, 15.9), turned to 90 degrees
- moved R2 111.8 mm to (-19.1, 18.5), turned to 90 degrees
- moved R28 110.5 mm to (-25.4, 19.8), turned to 90 degrees
- moved C9 109.4 mm to (-29.2, 21.0), turned to 90 degrees
- moved R1 106.4 mm to (-19.1, 22.3), turned to 90 degrees
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
Commit message: pcb work
Parts:
- added C29: (no value), Passive Components > Capacitors > Multilayer Ceramic Capacitors MLCC:0603_WAVE
- added D5: SML-D12, Opto-electronics > LED Emitters:0603_LED
- added M1: HM-11, Embedded > BLE Module:HM-11
- added R48: (no value), Passive Components > Resistors > Chip Resistors:0603_WAVE
- moved SW1 25.0 mm to (93.6, 83.4), turned to 0 degrees
- moved D2 15.0 mm to (86.5, 14.3), turned to 0 degrees
- moved D3 13.7 mm to (86.6, 16.7), turned to 180 degrees
- moved Q4 4.12 mm to (93.4, 92.7)
Connections:
- net RXD renamed USB-RX
- net TXD renamed USB-TX
- new net BLE-!RST: M1.11
- new net BLE-KEY: M1.16
- new net BLE-RX: M1.4
- new net BLE-TX: M1.2
- new net N$35: D5.P$2, R48.P$2
- new net N$36: M1.15, R48.P$1
- new net USB-SUS: U$5.17
- new net USB-WKUP: U$5.11
- net 3.3V: now also C29.P$1, M1.9
- net BTN_1: now also C20.P$2
- net BTN_2: now also C21.P$2
- net BTN_3: now also C22.P$2
- net BTN_4: now also C23.P$2
- net BTN_5: now also C24.P$2
- net GND: now also C29.P$2, D5.P$1, M1.12
- net N$12: no longer C23.P$2
- net N$14: no longer C24.P$2
- net N$3: no longer C20.P$2
- net N$6: no longer C21.P$2
- net N$8: no longer C22.P$2
Other:
- outline, holes or cut-outs redrawn

Commit message: pcb work
Parts:
- removed J5: 2EDG-2P, Connectors > Other:2EDG-2P
- added C30, C31, C32, C34, C35: 100n, Passive Components > Capacitors > Multilayer Ceramic Capacitors MLCC:0603_WAVE
- added C33, C36: 10u, Passive Components > Capacitors > Tantalum Capacitors:EIA3216
- added C37, C38: (no value), Passive Components > Capacitors > Multilayer Ceramic Capacitors MLCC:0603_WAVE
- added D6, D8: SK54L, Semiconductors > Discrete Semiconductors > Diodes & Rectifiers > Schottky Diodes & Rectifiers:DO214AA
- added D7: SML-D12, Opto-electronics > LED Emitters:0603_LED
- added J10, J11: 4P-PC-FAN, Thermal Management > Fans & Blowers:KF2510-3+1P
- added J12, J13: PCC-SMP, Connectors > Other:PCC-SMP
- added J2: 3X1_2.54, Connectors > Header:3X1_2.54
- added KK1: SK104, Thermal Management > Heatsinks:SK104
- added L1, L2: 68uH, Passive Components > Inductors, Chokes & Coils:1207
- added Q10, Q11, Q12, Q6, Q7, Q8, Q9: BC817-40, Semiconductors > Discrete Semiconductors > Transistors > Bipolar Transistors - BJT:SOT-23-3
- added Q5: MOC3051, Opto-electronics > Optocouplers\Photocouplers:DIP-6-SMD
- added R45, R46, R47, R49: (no value), Passive Components > Resistors > Chip Resistors:_1206
- added R50, R51: 54.9k, Passive Components > Resistors > Chip Resistors:_1206
- added R52, R60, R61, R62, R63, R64, R65, R66, R67, R68, R69, R70, R71, R72, R73, R74, R75, R76, R77, R78, R79, R80, R81, R82, R83, R84, R85: (no value), Passive Components > Resistors > Chip Resistors:0603_WAVE
- added R53, R59: 1.2k, Passive Components > Resistors > Chip Resistors:0603_WAVE
- added R54, R55: 10M, Passive Components > Resistors > Chip Resistors:0603_WAVE
- added R56, R57: 10k, Passive Components > Resistors > Chip Resistors:0603_WAVE
- added R58: 3.01k, Passive Components > Resistors > Chip Resistors:0603_WAVE
- added U$7: HLK-PM01, Power > AC\DC Converters:HLK-PM01
- added U$8: BTA16, Semiconductors > Discrete Semiconductors > Thyristors > Triacs:TO220DS
- added U8, U9: MIC4682, Power > Switching Controllers:SOIC8
- C15: value 1u -> 100n
- C16: value 1u -> 10u; device Passive Components > Capacitors > Multilayer Ceramic Capacitors MLCC:0603_WAVE -> Passive Components > Capacitors > Tantalum Capacitors:EIA3216
- C17: value (none) -> 100n
- C9: value (none) -> 10u; device Passive Components > Capacitors > Multilayer Ceramic Capacitors MLCC:0603_WAVE -> Passive Components > Capacitors > Tantalum Capacitors:EIA3216
- J4: value 2EDG-2P -> MICROSD; device Connectors > Other:2EDG-2P -> Connectors > card socket:MICRO-SD
- J7: value 2EDG-2P -> 3X1_2.54; device Connectors > Other:2EDG-2P -> Connectors > Header:3X1_2.54
- R36: value (none) -> 3.01k
- R40, R41: value (none) -> 54.9k; device Passive Components > Resistors > Chip Resistors:0603_WAVE -> Passive Components > Resistors > Chip Resistors:_1206
- R42: value (none) -> 10k
- moved C19 247.9 mm to (141.0, -87.0)
- moved C18 240.8 mm to (125.0, -87.0)
- moved C17 238.3 mm to (115.0, -87.0)
- moved J4 235.8 mm to (-97.0, -147.0)
- moved C25 207.3 mm to (-103.0, -136.0), turned to 0 degrees
- moved D5 191.5 mm to (97.0, 98.0), turned to 180 degrees
- moved C1 191.2 mm to (91.0, -87.0)
- moved C12 190.4 mm to (137.0, -87.0)
- moved C2 189.9 mm to (95.0, -87.0)
- moved C3 188.7 mm to (99.0, -87.0)
- moved C4 187.8 mm to (103.0, -87.0)
- moved C5 187.2 mm to (107.0, -87.0)
- moved C6 186.7 mm to (111.0, -87.0)
- moved C9 184.2 mm to (120.0, -87.0)
- moved R36 178.3 mm to (-3.00, -88.0)
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Connections:
- removed net SERVO-SIG: J8.P$1
- new net 12V: C13.P$1, C14.AN, C30.P$1, C34.P$1, F1.P$1, J10.2, J11.2, R1.P$2, R54.P$2, R55.P$2, R60.P$2, R71.P$2, R73.P$2, R82.P$2, U8.5, U9.5
- new net 12V-FB: C25.P$1, R82.P$1, R83.P$2
- new net 2.8V: C1.P$1, C12.P$1, C16.+, C18.P$1, C19.P$1, C2.P$1, C26.P$1, C29.P$1, C3.P$1, C32.P$1, C4.P$1, C5.P$1, C6.P$1, J1.1, J4.4, M1.9, R10.P$2, R11.P$2, R12.P$2, R13.P$2, R14.P$2, R18.P$2, R22.P$2, R28.P$2, R34.P$1, R35.P$1, R42.P$2, R44.P$2, R5.P$2, R6.P$2, R7.P$2, R8.P$2, R84.P$2, R85.P$2, R9.P$2, U$5.5, U1.24, U1.27, U1.38, U1.39, U1.55, U1.7, U2.8, U3.3, U4.8, U5.35, U5.40, U5.41, U5.42, U5.7, U5.8, U5.9, U7.16, U7.8
- new net 3.6V: C15.P$1, C31.P$1, C33.+, L1.2, R36.P$2, R78.P$2, U3.1
- new net 3.6V-FB: C38.P$1, R78.P$1, R79.P$2
- new net 5V-FB: C37.P$1, R80.P$1, R81.P$2
- new net AC-L: J3.P$2, J6.P$1, R40.1, U$7.AC2
- new net AC-N: J3.P$1, R50.1, U$7.AC1, U$8.A1
- new net FAN0-CTRL: R70.P$1
- new net FAN0-GND: R68.P$1
- new net FAN0-SNSE: R74.P$1, R75.P$2
- new net FAN1-CTRL: R72.P$1
- new net FAN1-GND: R69.P$1
- new net FAN1-SNSE: R76.P$1, R77.P$2
- new net N$34: Q5.P$1, R52.P$1
- new net N$37: Q5.P$4, R45.1
- new net N$38: Q5.P$6, R47.1
- new net N$39: R45.2, R46.1
- new net N$40: R47.2, R49.1
- new net N$41: J6.P$2, R46.2, U$8.A2
- new net N$42: R49.2, U$8.G
- new net N$43: R36.P$1, R53.P$2, U9.1
- new net N$44: R54.P$1, R57.P$2, U9.3
- new net N$45: D6.C, L2.1, U8.8
- new net N$46: R58.P$1, R59.P$2, U8.1
- new net N$47: R55.P$1, R56.P$2, U8.3
- new net N$48: C28.P$1, U$5.6
- new net N$49: Q6.P$1, R62.P$2
- new net N$50: J2.P$1, Q6.P$3, R63.P$1
- new net N$51: D7.P$2, R61.P$2
- new net N$52: J7.P$1, Q7.P$3, R65.P$1
- new net N$53: Q7.P$1, R64.P$2
- new net N$54: Q8.P$1, R66.P$2
- new net N$55: J8.P$1, Q8.P$3, R67.P$1
- new net N$56: Q9.P$1, R68.P$2
- new net N$57: J11.1, Q9.P$3
- new net N$58: Q10.P$1, R70.P$2
- new net N$59: J11.4, Q10.P$3, R71.P$1
- new net N$60: Q11.P$1, R69.P$2
- new net N$61: Q12.P$1, R72.P$2
- new net N$62: J10.4, Q12.P$3, R73.P$1
- new net N$63: J10.1, Q11.P$3
- new net N$64: J11.3, R74.P$2
- new net N$65: J10.3, R76.P$2
- new net N$67: J4.2, R85.P$1
- new net SD-CD: J4.9, R84.P$1
- new net SERVO0-SIG: R62.P$1
- new net SERVO1-SIG: R66.P$1
- new net SERVO2-SIG: R64.P$1
- new net USB-RST: U$5.9
- new net V_USB: C27.P$1, D4.4, R37.P$2, U$5.7, U$6.VBUS
- net 3.3V: no longer C1.P$1, C12.P$1, C16.P$1, C17.P$1, C18.P$1, C19.P$1, C2.P$1, C25.P$1, C26.P$1, C27.P$1, C28.P$1, C29.P$1, C3.P$1, C4.P$1, C5.P$1, C6.P$1, J1.1, M1.9, R10.P$2, R11.P$2, R12.P$2, R13.P$2, R14.P$2, R18.P$2, R22.P$2, R28.P$2, R34.P$1, R35.P$1, R36.P$1, R42.P$2, R44.P$2, R5.P$2, R6.P$2, R7.P$2, R8.P$2, R9.P$2, U$5.5, U$5.6, U$5.7, U1.24, U1.27, U1.38, U1.39, U1.55, U1.7, U2.8, U3.3, U4.8, U5.1, U5.35, U5.40, U5.41, U5.42, U5.7, U5.8, U5.9, U7.16, U7.8
- net 5V: now also C35.P$1, C36.+, J2.P$2, J7.P$2, L2.2, R52.P$2, R58.P$2, R61.P$1, R63.P$2, R65.P$2, R67.P$2, R80.P$2, U5.1; no longer B1.1, C13.P$1, C14.AN, C15.P$1, F1.P$1, J6.P$1, R1.P$2, U3.1
- net GND: now also C16.-, C30.P$2, C31.P$2, C32.P$2, C33.-, C34.P$2, C35.P$2, C36.-, C37.P$2, C38.P$2, C9.-, D6.A, D8.A, J12.3-BAR, J12.4-BAR, J13.3-BAR, J13.4-BAR, J2.P$3, J4.6, J4.BODY1, J4.BODY2, J4.BODY3, J4.BODY4, J7.P$3, Q10.P$2, Q11.P$2, Q12.P$2, Q6.P$2, Q7.P$2, Q8.P$2, Q9.P$2, R53.P$1, R56.P$1, R57.P$1, R59.P$1, R75.P$1, R77.P$1, R79.P$1, R81.P$1, R83.P$1, U$7.-VO, U8.2, U8.4, U8.6, U8.7, U9.2, U9.4, U9.6, U9.7; no longer C16.P$2, C9.P$2, J3.P$2
- net N$20: now also R40.2, R41.1; no longer J7.P$1, R40.P$1
- net N$21: now also R41.2; no longer R40.P$2
- net N$28: now also D8.C, L1.1, U9.8; no longer R36.P$2, U$5.9
- net N$29: now also R51.2; no longer R41.P$2
- net N$30: now also R50.2, R51.1; no longer J7.P$2, R41.P$1
- net N$31: now also U$7.+VO; no longer J3.P$1
- net N$4: now also B1.1, R60.P$1; no longer D4.4, R37.P$2, U$6.VBUS
- net N$7: now also D7.P$1, Q5.P$2; no longer J6.P$2
- net N$9: now also C17.P$1, C9.+; no longer C9.P$1
- net TC_VIN0+: now also J12.1-T+; no longer J4.P$1
- net TC_VIN0-: now also J12.2-T-; no longer J4.P$2
- net TC_VIN1+: now also J13.1-T+; no longer J5.P$1
- net TC_VIN1-: now also J13.2-T-; no longer J5.P$2
Routing:
- net AC-L: track 0.00 -> 63.7 mm
- net AC-N: track 0.00 -> 49.9 mm
- net N$41: track 0.00 -> 31.0 mm
- net N$42: track 0.00 -> 20.0 mm
- net N$37: track 0.00 -> 18.3 mm
- net N$29: track 0.00 -> 8.44 mm
- net N$38: track 0.00 -> 4.82 mm
- net N$40: track 0.00 -> 4.00 mm
- net N$39: track 0.00 -> 4.00 mm
- net N$21: track 0.00 -> 3.70 mm
- net N$20: track 0.00 -> 3.50 mm
- net N$30: track 0.00 -> 3.45 mm
Other:
- outline, holes or cut-outs redrawn

Commit message: pn532 dev
Parts:
- removed C15, C32: 100n, Passive Components > Capacitors > Multilayer Ceramic Capacitors MLCC:0603_WAVE
- removed U3: MIC39100, Power > LDO Voltage Regulators:SOT230P700X180-4N
- moved J4 290.7 mm to (70.0, 91.0), turned to 180 degrees
- moved C16 150.4 mm to (-103.0, -166.0), turned to 0 degrees
- moved Q5 1.00 mm to (56.0, 17.0)
Connections:
- net 2.8V: now also U1.46; no longer C32.P$1, U3.3
- net 3.6V: no longer C15.P$1, U3.1
- net 5V: now also U1.45
- net GND: no longer C15.P$2, C32.P$2, U3.2, U3.4
Routing:
- net N$38: track 4.82 -> 5.82 mm
Other:
- outline, holes or cut-outs redrawn

Commit message: pcb work
Parts:
- removed B2, B3, B4, B5, B6: PUSH-SILENT, Eletromechanical > Switches > Tactile Switches:SILENT_BUT
- removed C30, C31: 100n, Passive Components > Capacitors > Multilayer Ceramic Capacitors MLCC:0603_WAVE
- removed C33, C36: 10u, Passive Components > Capacitors > Tantalum Capacitors:EIA3216
- removed C37, C38: (no value), Passive Components > Capacitors > Multilayer Ceramic Capacitors MLCC:0603_WAVE
- removed D1: WS2812B, Opto-electronics > LED Emitters:WS2812B
- removed J8: 3X1_2.54, Connectors > Header:3X1_2.54
- removed J9: 2X1_2.54, Connectors > Header:2X1_2.54
- removed Q2, Q8: BC817-40, Semiconductors > Discrete Semiconductors > Transistors > Bipolar Transistors - BJT:SOT-23-3
- removed R12, R13, R19, R20, R21, R22, R23, R25, R26, R27, R28, R29, R3, R30, R31, R32, R33, R4, R43, R44, R66, R67, R78, R79, R80, R81, R85: (no value), Passive Components > Resistors > Chip Resistors:0603_WAVE
- removed R36: 3.01k, Passive Components > Resistors > Chip Resistors:0603_WAVE
- removed R53: 1.2k, Passive Components > Resistors > Chip Resistors:0603_WAVE
- removed R54: 10M, Passive Components > Resistors > Chip Resistors:0603_WAVE
- removed R57: 10k, Passive Components > Resistors > Chip Resistors:0603_WAVE
- removed U9: MIC4682, Power > Switching Controllers:SOIC8
- added C15: 100n, Passive Components > Capacitors > Multilayer Ceramic Capacitors MLCC:0603_WAVE
- added C32: (no value), Passive Components > Capacitors > Multilayer Ceramic Capacitors MLCC:0603_WAVE
- added D10, D11, D12, D9: WS2812B, Opto-electronics > LED Emitters:3535
- added J5: 2X1_2.54, Connectors > Header:2X1_2.54
- added U11: 74HC123, Semiconductors > Integrated Circuits - ICs > Logic ICs > Logic Gates:TSSOP-16
- added U12: 74LVC1G08, Semiconductors > Integrated Circuits - ICs > Logic ICs > Logic Gates:SC-70-5
- added U13: 74LVC1G32, Semiconductors > Integrated Circuits - ICs > Logic ICs > Logic Gates:SC-70-5
- C1, C18, C2, C20, C3, C4, C5, C6, C7: value (none) -> 100n
- C13: value 100n -> (none); device Passive Components > Capacitors > Multilayer Ceramic Capacitors MLCC:0603_WAVE -> Passive Components > Capacitors > Aluminium Electrolytic Capacitors:PANASONIC_D
- C14: device Passive Components > Capacitors > Aluminium Electrolytic Capacitors:10X10-EL -> Passive Components > Capacitors > Aluminium Electrolytic Capacitors:PANASONIC_D
- C16: value 10u -> (none); device Passive Components > Capacitors > Tantalum Capacitors:EIA3216 -> Passive Components > Capacitors > Multilayer Ceramic Capacitors MLCC:0603_WAVE
- C17: value 100n -> 1u
- C21: value (none) -> 4u7
- C22, C23: value (none) -> 100p
- C24: value (none) -> 1u
- C35: value 100n -> (none)
- C9: value 10u -> 1u; device Passive Components > Capacitors > Tantalum Capacitors:EIA3216 -> Passive Components > Capacitors > Multilayer Ceramic Capacitors MLCC:0603_WAVE
- D8: value SK54L -> WS2812B; device Semiconductors > Discrete Semiconductors > Diodes & Rectifiers > Schottky Diodes & Rectifiers:DO214AA -> Opto-electronics > LED Emitters:3535
- L1: value 68uH -> 4.7nH; device Passive Components > Inductors, Chokes & Coils:1207 -> Passive Components > Inductors, Chokes & Coils:0805
- R14, R15: value (none) -> 3k95
- R59: value 1.2k -> 1k
- U1: value EFM32GG11B8XX_Q64 -> EFM32GG11B8XX_Q100; device Semiconductors > Embedded Processors & Controllers > Microcontrollers - MCU:QFP64 -> Semiconductors > Embedded Processors & Controllers > Microcontrollers - MCU:QFP100
- moved R84 319.8 mm to (72.0, 109.0), turned to 90 degrees
- moved C16 296.8 mm to (86.8, 62.2), turned to 270 degrees
- moved C25 237.6 mm to (37.0, 56.0), turned to 90 degrees
- moved R83 236.2 mm to (39.0, 56.0), turned to 270 degrees
- moved R82 234.3 mm to (41.0, 56.0), turned to 90 degrees
- moved D8 216.5 mm to (87.8, 92.2), flipped to the bottom, turned to 0 degrees
- moved R77 212.5 mm to (74.5, 53.5), turned to 270 degrees
- moved C19 209.5 mm to (67.0, 109.0)
- moved U8 209.0 mm to (49.5, 49.0), turned to 270 degrees
- moved C12 208.8 mm to (65.0, 109.0)
- moved C1 207.6 mm to (65.0, 119.0)
- moved C18 207.6 mm to (99.0, 119.0)
- moved C2 207.6 mm to (69.0, 119.0)
- moved C26 207.6 mm to (49.0, 119.0)
- moved C3 207.6 mm to (73.0, 119.0)
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Connections:
- removed net 3.6V: C31.P$1, C33.+, L1.2, R36.P$2, R78.P$2
- removed net 3.6V-FB: C38.P$1, R78.P$1, R79.P$2
- removed net 5V-FB: C37.P$1, R80.P$1, R81.P$2
- removed net BLE-RX: M1.4
- removed net BLE-TX: M1.2
- removed net BTN_1: C20.P$2, R30.P$2
- removed net BTN_2: C21.P$2, R15.P$2
- removed net BTN_3: C22.P$2, R31.P$2
- removed net BTN_4: C23.P$2, R32.P$2
- removed net BTN_5: C24.P$2, R33.P$2
- removed net DOOR-SWITCH: R43.P$2
- removed net LED_DI: R4.P$1
- removed net N$11: D1.4, Q2.P$3, R3.P$1
- removed net N$27: R20.P$2, U4.4
- removed net N$28: D8.C, L1.1, U9.8
- removed net N$3: B2.P$2, R10.P$1, R30.P$1
- removed net N$32: J9.2
- removed net N$33: J9.1, R43.P$1, R44.P$1
- removed net N$43: R36.P$1, R53.P$2, U9.1
- removed net N$44: R54.P$1, R57.P$2, U9.3
- removed net N$54: Q8.P$1, R66.P$2
- removed net N$55: J8.P$1, Q8.P$3, R67.P$1
- removed net N$67: J4.2, R85.P$1
- removed net SD-CD: J4.9, R84.P$1
- removed net SERVO1-SIG: R66.P$1
- removed net US1-MISO-TFT: U5.33
- removed net US1-MOSI-TFT: U5.34
- removed net USB-WKUP: U$5.11
- removed net ZERO-CROSS: R42.P$1, U6.P$5
- new net !LED_CS: U11.1, U11.9
- new net DOOR-SW: C16.P$1, R11.P$2
- new net LED_MOSI: U12.2
- new net LED_SCK: U11.10, U12.1
- new net N$69: U11.5, U13.1
- new net N$77: U11.13, U13.2
- new net N$78: U11.2, U12.4
- new net N$79: C22.P$2, R14.P$2, U11.15
- new net N$80: C22.P$1, U11.14
- new net N$81: C23.P$2, R15.P$2, U11.7
- new net N$82: C23.P$1, U11.6
- new net SDIO-CD: J4.9, R84.P$1, U1.86
- new net SDIO-CLK: J4.5, U1.97
- new net SDIO-CMD: J4.3, U1.96
- new net SDIO-DAT0: J4.7, U1.95
- new net SDIO-DAT1: J4.8, U1.94
- new net SDIO-DAT2: J4.1, U1.93
- new net SDIO-DAT3: J4.2, U1.92
- new net U1RX-BLE-TX: M1.2, U1.63
- new net U1TX-BLE-RX: M1.4, U1.62
- new net US0-MISO-TFT: U1.19, U5.33
- new net US0-MOSI-TFT: U1.18, U5.34
- new net WTIM1-CC1-ZERO-CROSS: R42.P$1, U1.64, U6.P$5
- net !RESET: now also U1.36; no longer U1.20
- net 12V: now also C13.+; no longer C13.P$1, C14.AN, C30.P$1, R54.P$2, U9.5
- net 12V-FB: now also U1.45
- net 2.8V: now also C10.P$1, C11.P$1, C20.P$1, C24.P$1, C7.P$1, C8.P$1, U1.17, U1.31, U1.41, U1.44, U1.57, U1.73, U1.8, U1.82; no longer C16.+, R11.P$2, R12.P$2, R13.P$2, R14.P$2, R22.P$2, R28.P$2, R44.P$2, R85.P$2, U1.24, U1.27, U1.38, U1.39, U1.46, U1.55, U1.7
- net 3.3V: now also U12.5; no longer C10.P$1, C11.P$1, C8.P$1
- net 5V: now also C14.+, C15.P$1, C32.P$1, C9.P$1, D10.3, D11.3, D12.3, D8.3, D9.3, R14.P$1, R15.P$1, U1.72, U1.79, U11.11, U11.16, U11.3, U13.5; no longer C36.+, C7.P$1, D1.1, J8.P$2, R3.P$2, R67.P$2, R80.P$2, U1.45
- net GND: now also C13.-, C14.-, C15.P$2, C16.P$2, C20.P$2, C21.P$2, C24.P$2, C32.P$2, C9.P$2, D10.1, D11.1, D12.1, D8.1, D9.1, J5.2, U1.16, U1.32, U1.55, U1.59, U1.83, U11.8, U12.3, U13.3; no longer B2.P$1, B3.P$1, B4.P$1, B5.P$1, B6.P$1, C13.P$2, C14.CAT, C16.-, C20.P$1, C21.P$1, C22.P$1, C23.P$1, C24.P$1, C30.P$2, C31.P$2, C33.-, C36.-, C37.P$2, C38.P$2, C9.-, D1.3, D8.A, J8.P$3, Q2.P$2, Q8.P$2, R21.P$1, R23.P$1, R27.P$1, R29.P$1, R53.P$1, R57.P$1, R79.P$1, R81.P$1, U1.23, U1.36, U1.56, U1.8, U9.2, U9.4, U9.6, U9.7
- net I2C0-SCL-SENS: now also U1.52
- net I2C0-SDA-SENS: now also U1.51
- net I2C1-SCL-TFT: now also U1.23
- net I2C1-SDA-TFT: now also U1.22
- net MAIN_HFXTAL_N: now also U1.43
- net MAIN_HFXTAL_P: now also U1.42
- net MAIN_LFXTAL_N: now also U1.25
- net MAIN_LFXTAL_P: now also U1.24
- net N$1: now also J5.1, R10.P$1, R11.P$1; no longer R25.P$2, U7.2
- net N$10: now also D10.2, D9.4; no longer Q2.P$1, R4.P$2
- net N$12: now also D8.2, U13.4; no longer B5.P$2, R13.P$1, R32.P$1
- net N$14: now also L1.2, U1.56; no longer B6.P$2, R14.P$1, R33.P$1
- net N$2: now also D8.4, D9.2; no longer R26.P$2, U7.4
- net N$26: now also C21.P$1, L1.1, U1.58; no longer R19.P$2, U4.2
- net N$6: now also D10.4, D11.2; no longer B3.P$2, R11.P$1, R15.P$1
- net N$8: now also D11.4, D12.2; no longer B4.P$2, R12.P$1, R31.P$1
- net N$9: now also U1.60; no longer C9.+, U1.40
- net QSPI_CLK: now also U1.84
- net QSPI_CS0: now also U1.85
- net QSPI_D0: now also U1.88
- net QSPI_D1: now also U1.89
- net QSPI_D2: now also U1.90
- net QSPI_D3: now also U1.91
- net SWCLK: now also U1.76; no longer U1.49
- net SWDIO: now also U1.77; no longer U1.50
- net SWO: now also U1.78; no longer U1.51
- net TC_VIN0+: now also U4.2; no longer R19.P$1, R21.P$2, R22.P$1
- net TC_VIN0-: now also U4.4; no longer R20.P$1, R23.P$2
- net TC_VIN1+: now also U7.2; no longer R25.P$1, R27.P$2, R28.P$1
- net TC_VIN1-: now also U7.4; no longer R26.P$1, R29.P$2
- net USB-RX: now also U1.4
- net USB-TX: now also U1.5
Routing:
- net 12V: track 0.00 -> 100.3 mm, vias 0 -> 1
- net 5V: track 0.00 -> 98.0 mm, vias 0 -> 5
- net AC-L: track 63.7 -> 34.7 mm
- net N$64: track 0.00 -> 21.4 mm, vias 0 -> 1
- net N$59: track 0.00 -> 20.8 mm
- net !LED_CS: track 0.00 -> 19.7 mm, vias 0 -> 2
- net N$45: track 0.00 -> 19.5 mm
- net LED_SCK: track 0.00 -> 17.4 mm
- net N$65: track 0.00 -> 17.4 mm, vias 0 -> 1
- net N$69: track 0.00 -> 15.8 mm, vias 0 -> 2
- net N$62: track 0.00 -> 14.8 mm
- net N$57: track 0.00 -> 13.8 mm
- net N$7: track 0.00 -> 13.2 mm
- net N$50: track 0.00 -> 11.3 mm
- net N$52: track 0.00 -> 10.9 mm
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- added copper zone on layer 1, net AC-L
Other:
- outline, holes or cut-outs redrawn

Commit message: sync
Parts:
- added JP1, JP2: JUMPER-SMT_3_1-NC_PASTE_SILK, Utility > Board:SMT-JUMPER_3_1-NC_PASTE_SILK
- moved C20 105.3 mm to (28.5, 95.5), turned to 90 degrees
- moved C7 101.0 mm to (25.0, 95.5), turned to 90 degrees
- moved C14 27.2 mm to (47.0, 45.0), turned to 90 degrees
- moved R59 17.3 mm to (59.5, 41.0), turned to 180 degrees
- moved C34 14.8 mm to (57.5, 32.5)
- moved R55 14.8 mm to (51.5, 34.5)
- moved R56 14.8 mm to (51.5, 38.5)
- moved U8 14.8 mm to (57.5, 36.5)
- moved R58 13.1 mm to (55.5, 41.0), turned to 180 degrees
- moved C13 12.0 mm to (62.5, 27.5), turned to 180 degrees
- moved C15 12.0 mm to (51.5, 43.5), turned to 270 degrees
- moved D6 11.7 mm to (63.2, 35.5), turned to 270 degrees
- moved U$5 10.7 mm to (40.9, 86.7), turned to 0 degrees
- moved R2 8.19 mm to (35.3, 56.4), turned to 180 degrees
- moved D7 7.91 mm to (64.0, 21.0)
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- renumbered U$6 to J8
Connections:
- net I2C1-SCL-TFT renamed I2C1-SCL-TTFT
- net I2C1-SDA-TFT renamed I2C1-SDA-TTFT
- net USB-RX renamed U0TX-USB-RX
- net USB-TX renamed U0RX-USB-TX
- removed net !LED_CS: U11.1, U11.9
- removed net !TFT-IRQ: U5.46
- removed net !TFT-RST: U5.47
- removed net FAN0-CTRL: R70.P$1
- removed net FAN0-GND: R68.P$1
- removed net FAN0-SNSE: R74.P$1, R75.P$2
- removed net FAN1-CTRL: R72.P$1
- removed net FAN1-GND: R69.P$1
- removed net FAN1-SNSE: R76.P$1, R77.P$2
- removed net LED_MOSI: U12.2
- removed net LED_SCK: U11.10, U12.1
- removed net SERVO0-SIG: R62.P$1
- removed net SERVO2-SIG: R64.P$1
- removed net SSR-OUT: R39.P$1
- removed net TIM3_CC2_BUZZ: R2.P$1
- removed net UART-D+: D4.3, J8.D+, U$5.3
- removed net UART-D-: D4.2, J8.D-, U$5.4
- removed net US0-MISO-TFT: U1.19, U5.33
- removed net US0-MOSI-TFT: U1.18, U5.34
- removed net WTIM2_CC1_TFT_BL: R24.P$1
- new net !LED-CS: U1.66, U11.1, U11.9
- new net !TTFT-IRQ: U1.12, U5.46
- new net !TTFT-RST: U1.15, U5.47
- new net PRS-CH11-SSR-OUT: R39.P$1, U1.50
- new net TIM0-CC0-BUZZ: R2.P$1, U1.27
- new net TIM1-CC0-TFT-BL: R24.P$1, U1.9
- new net TIM2-CC2FAN0-SNSE: R74.P$1, R75.P$2, U1.70
- new net TIM3-CC0-FAN1-SNSE: R76.P$1, R77.P$2, U1.7
- new net TIM5-CC0-FAN0-GND: R68.P$1, U1.68
- new net TIM5-CC1-FAN0-CTRL: R70.P$1, U1.69
- new net TIM6-CC0-FAN1-GND: R69.P$1, U1.46
- new net TIM6-CC1-FAN1-CTRL: R72.P$1, U1.47
- new net US0-LED-MOSI: U1.67, U12.2
- new net US0-LED-SCK: U1.65, U11.10, U12.1
- new net US1-MISO-TFT: U1.20, U5.33
- new net US1-MOSI-TFT: U1.19, U5.34
- new net USB-D+: D4.3, J8.VBUS, JP1.1, JP1.2, U1.75
- new net USB-D-: D4.2, J8.D+, JP2.1, JP2.2, U1.74
- new net USB-ID: J8.ID, U1.80
- new net USB-UART-D+: JP1.3, U$5.3
- new net USB-UART-D-: JP2.3, U$5.4
- new net WTIM0-CC0-ZERO-CROSS: U1.64
- new net WTIM2-CC0-SERVO0-SIG: R62.P$1, U1.48
- new net WTIM2-CC1-SERVO1-SIG: R64.P$1, U1.49
- net !TFT_RESET: now also U1.14
- net BLE-!RST: now also U1.53
- net BLE-KEY: now also U1.61
- net DOOR-SW: now also U1.54
- net TFT-DC: now also U1.26
- net US1-CLK-TFT: now also U1.21
- net US1-CS-TFT: now also U1.18
- net USB-RST: now also U1.3
- net USB-SUS: now also U1.2
- net V_USB: now also J8.D-; no longer J8.VBUS
- net WTIM1-CC1-ZERO-CROSS: no longer U1.64
Routing:
- net 12V: track 100.3 -> 60.8 mm, vias 1 -> 0
- net US1-CS-TFT: track 1.78 -> 22.9 mm
- net !LED_CS: track 19.7 -> 0.00 mm, vias 2 -> 0
- net !LED-CS: track 0.00 -> 19.7 mm, vias 0 -> 2
- net US0-LED-SCK: track 0.00 -> 17.4 mm
- net LED_SCK: track 17.4 -> 0.00 mm
- net US0-LED-MOSI: track 0.00 -> 9.05 mm
- net LED_MOSI: track 9.05 -> 0.00 mm
- net N$17: track 5.20 -> 0.26 mm
- net 5V: track 98.0 -> 100.9 mm, vias 5 -> 4
- net N$45: track 19.5 -> 17.5 mm
- net TIM3-CC0-FAN1-SNSE: track 0.00 -> 1.85 mm
- net TIM2-CC2FAN0-SNSE: track 0.00 -> 1.85 mm
- net FAN1-SNSE: track 1.85 -> 0.00 mm
- net FAN0-SNSE: track 1.85 -> 0.00 mm
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Other:
- outline, holes or cut-outs redrawn
