File: pcb/r3eflow-v3.brd (EAGLE design)
At the start: 100 x 100 mm, 143 parts, among them J1 SH-6, J10 4P-PC-FAN, J11 4P-PC-FAN, J12 PCC-SMP, J13 PCC-SMP, J2 3X1_2.54, J3 2EDG-2P, J4 MICROSD, J5 2X1_2.54, J6 2EDG-2P, J7 3X1_2.54, J8 USB-SHIELD, M1 HM-11, Q1 BC817-40, Q10 BC817-40, Q11 BC817-40, Q12 BC817-40, Q3 BC817-40, Q4 BC817-40, Q5 MOC3051, Q6 BC817-40, Q7 BC817-40, Q9 BC817-40, U1 EFM32GG11B8XX_Q100, U11 74HC123, U12 74LVC1G08, U13 74LVC1G32, U2 SST26VF064B, U4 MCP9600, U5 ER-TFT035-6BOT, U6 H11AA1, U7 MCP9600, U8 MIC4682, Y1 32.768KHz, Y2 8MHz

Commit message: pcb work
Parts:
- removed C1, C18, C2, C20, C3, C4, C5, C6, C7: 100n, Passive Components > Capacitors > Multilayer Ceramic Capacitors MLCC:0603_WAVE
- removed C10, C11, C12, C19, C25, C26, C27, C28, C29, C8: (no value), Passive Components > Capacitors > Multilayer Ceramic Capacitors MLCC:0603_WAVE
- removed C13: (no value), Passive Components > Capacitors > Aluminium Electrolytic Capacitors:PANASONIC_D
- removed C17, C24, C9: 1u, Passive Components > Capacitors > Multilayer Ceramic Capacitors MLCC:0603_WAVE
- removed C21: 4u7, Passive Components > Capacitors > Multilayer Ceramic Capacitors MLCC:0603_WAVE
- removed D2, D3, D5, D7: SML-D12, Opto-electronics > LED Emitters:0603_LED
- removed D4: SP0503BAHT, Circuit Protection > ESD Suppressors \ TVS Diodes:SOT143
- removed J8: USB-SHIELD, Connectors > USB:USB-M-S1
- removed JP1, JP2: JUMPER-SMT_3_1-NC_PASTE_SILK, Utility > Board:SMT-JUMPER_3_1-NC_PASTE_SILK
- removed L1: 4.7nH, Passive Components > Inductors, Chokes & Coils:0805
- removed R1, R18, R34, R35, R5, R52, R6, R60, R61, R7, R82, R83, R84: (no value), Passive Components > Resistors > Chip Resistors:0603_WAVE
- removed R37: 22.1k, Passive Components > Resistors > Chip Resistors:0603_WAVE
- removed R38: 47.5k, Passive Components > Resistors > Chip Resistors:0603_WAVE
- removed R47, R49: (no value), Passive Components > Resistors > Chip Resistors:_1206
- removed SW1: (no value), Eletromechanical > Switches > Tactile Switches:PUSH_BUTTON
- removed U$5: CP2102N, Semiconductors > Integrated Circuits - ICs > Interface ICs > USB Interface IC:QFN24
- removed U13: 74LVC1G32, Semiconductors > Integrated Circuits - ICs > Logic ICs > Logic Gates:SC-70-5
- removed Y1: 32.768KHz, Passive Components > Frequency Control & Timing Devices > Crystals:CM200S
- removed Y2: 8MHz, Passive Components > Frequency Control & Timing Devices > Crystals:2-SMD-5X3
- added C101, C102, C103, C104, C105, C110, C111: 100n, Passive Components > Capacitors > Multilayer Ceramic Capacitors MLCC:0603_WAVE
- added C106, C108, C109: 1u, Passive Components > Capacitors > Multilayer Ceramic Capacitors MLCC:0603_WAVE
- added C107: 4u7, Passive Components > Capacitors > Multilayer Ceramic Capacitors MLCC:0603_WAVE
- added C205, C206, C207, C208, C209, C301, C302, C403: (no value), Passive Components > Capacitors > Multilayer Ceramic Capacitors MLCC:0603_WAVE
- added C402: (no value), Passive Components > Capacitors > Aluminium Electrolytic Capacitors:PANASONIC_D
- added D206: SP0503BAHT, Circuit Protection > ESD Suppressors \ TVS Diodes:SOT143
- added D207, D208, D209, D301: LED0603, Opto-electronics > LED Emitters:CHIPLED_0603
- added J201: USB-SHIELD, Connectors > USB:USB-M-S1
- added JP201, JP202: JUMPER-SMT_3_1-NC_PASTE_SILK, Utility > Board:SMT-JUMPER_3_1-NC_PASTE_SILK
- added L101: 4.7nH, Passive Components > Inductors, Chokes & Coils:_0805
- added LOGO101: DESIGNEDINPT, Utility > Silkscreen:DESIGNEDINPT
- added LOGO102: RAFAEL_SILVA, Utility > Silkscreen:RAFAEL_SILVA_5MM_ALT_3
- added LOGO103: OSHW-LOGOL, Utility > Silkscreen:OSHW-LOGO-L
- added R101, R102, R105, R106, R206, R209, R210, R213, R214, R306, R307, R405, R406: (no value), Passive Components > Resistors > Chip Resistors:0603_WAVE
- added R207: 22.1k, Passive Components > Resistors > Chip Resistors:0603_WAVE
- added R208: 47.5k, Passive Components > Resistors > Chip Resistors:0603_WAVE
- added R313, R315: (no value), Passive Components > Resistors > Chip Resistors:_1206
- added SW101: (no value), Eletromechanical > Switches > Tactile Switches:PUSH_BUTTON
- added TP1, TP10, TP11, TP12, TP13, TP14, TP15, TP16, TP17, TP18, TP19, TP2, TP20, TP201, TP202, TP21, TP22, TP26, TP3, TP301, TP302, TP4, TP5, TP6, TP7, TP8, TP9: TEST_POINT, Utility > Board:TEST_POINT
- added U203: 74LVC1G32, Semiconductors > Integrated Circuits - ICs > Logic ICs > Logic Gates:SC-70-5
- added U205: CP2102N, Semiconductors > Integrated Circuits - ICs > Interface ICs > USB Interface IC:QFN24
- added Y101: 8MHz, Passive Components > Frequency Control & Timing Devices > Crystals:2-SMD-5X3
- added Y102: 32.768KHz, Passive Components > Frequency Control & Timing Devices > Crystals:CM200S
- renumbered B1 to B201, C14 to C404, C15 to C405, C16 to C303, C22 to C201, C23 to C202, C32 to C204, C34 to C401, C35 to C203, D10 to D203, D11 to D204, D12 to D205, D6 to D401, D8 to D201, D9 to D202, F1 to F401, J1 to J102, J10 to J308, J11 to J306, J12 to J301, J13 to J304, J2 to J302, J3 to J401, J4 to J101, J5 to J307, J6 to J305, J7 to J303, KK1 to KK301, L2 to L401, M1 to M201, Q1 to Q202, Q10 to Q305, Q11 to Q308, Q12 to Q307, Q3 to Q201, Q4 to Q303, Q5 to Q304, Q6 to Q301, Q7 to Q302, Q9 to Q306, R10 to R326, R11 to R323, R14 to R201, R15 to R202, R16 to R204, R17 to R205, R2 to R212, R24 to R203, R39 to R305, R40 to R308, R41 to R310, R42 to R316, R45 to R312, R46 to R314, R48 to R211, R50 to R309, R51 to R311, R55 to R401, R56 to R402, R58 to R403, R59 to R404, R62 to R301, R63 to R302, R64 to R303, R65 to R304, R68 to R319, R69 to R325, R70 to R318, R71 to R321, R72 to R324, R73 to R328, R74 to R320, R75 to R317, R76 to R327, R77 to R322, R8 to R103, R9 to R104, U$7 to ACDC401, U$8 to D302, U1 to U101, U11 to U202, U12 to U201, U2 to U102, U4 to U301, U5 to U204, U6 to U303, U7 to U302, U8 to U401
Connections:
- net N$10 renamed D9-DO
- net N$2 renamed D8_DO
- net N$22 renamed TFT-LEDK1
- net N$23 renamed TFT-LEDK2
- net N$24 renamed TFT-LEDK
- net N$46 renamed 5V-FB
- net N$6 renamed D10-DO
- net N$79 renamed U11.1-RC
- net N$8 renamed D11-DO
- net N$80 renamed U11.1-C
- net N$81 renamed U11.2-RC
- net N$82 renamed U11.2-C
- net TC0-ALRT2 renamed U4-ALRT2
- net TC0-ALRT3 renamed U4-ALRT3
- net TC0-ALRT4 renamed U4-ALRT4
- net TC1-ALRT2 renamed U7-ALRT2
- net TC1-ALRT3 renamed U7-ALRT3
- net TC1-ALRT4 renamed U7-ALRT4
- removed net 3.3V: U201.5
- removed net N$12: D201.2, U13.4
- removed net N$14: L1.2, U101.56
- removed net N$26: C21.P$1, L1.1, U101.58
- removed net N$48: C28.P$1, U$5.6
- removed net N$9: C17.P$1, U101.60
- removed net TC0-ALRT1: U301.11
- removed net TC1-ALRT1: U302.11
- removed net WTIM0-CC0-ZERO-CROSS: U101.64
- new net D8-DI: D201.2, TP201.1, U203.4
- new net DECOUPLE: C109.P$1, U101.60
- new net DVDD: C107.P$1, L101.1, U101.58
- new net N$84: D206.3, J201.D+, JP202.2
- new net N$85: D206.2, J201.D-, JP201.2
- new net PA0: TP1.1, U101.1
- new net PA10: TP4.1, U101.29
- new net PA11: TP5.1, U101.30
- new net PA12: TP6.1, U101.33
- new net PA13: TP7.1, U101.34
- new net PA14: TP8.1, U101.35
- new net PA15: TP9.1, U101.100
- new net PA5: TP2.1, U101.6
- new net PA9: TP3.1, U101.28
- new net PB1: TP21.1, U101.10
- new net PB10: TP17.1, U101.38
- new net PB11: TP16.1, U101.39
- new net PB12: TP15.1, U101.40
- new net PB2: TP20.1, U101.11
- new net PB4: TP19.1, U101.13
- new net PB9: TP18.1, U101.37
- new net PC11: TP10.1, U101.71
- new net PE14: TP11.1, U101.98
- new net PE15: TP12.1, U101.99
- new net PF5: TP14.1, U101.81
- new net PF9: TP13.1, U101.87
- new net U4-ALRT1: TP22.1, U301.11
- new net U7-ALRT1: TP26.1, U302.11
- new net VREGSW: L101.2, U101.56
- net !RESET: now also SW101.1, SW101.2; no longer SW1.1, SW1.2
- net 12V: now also C402.+, R213.P$2, R214.P$2, R405.P$2; no longer C13.+, R1.P$2, R60.P$2, R82.P$2
- net 12V-FB: now also C403.P$1, R405.P$1, R406.P$2; no longer C25.P$1, R82.P$1, R83.P$2
- net 2.8V: now also C101.P$1, C102.P$1, C103.P$1, C104.P$1, C105.P$1, C106.P$1, C110.P$1, C111.P$1, C205.P$1, C206.P$1, C207.P$1, C208.P$1, C209.P$1, C301.P$1, C302.P$1, R101.P$2, R102.P$2, R105.P$2, R106.P$2, R206.P$2, R209.P$1, R210.P$1, U201.5, U205.5, U205.6, U205.7; no longer C1.P$1, C10.P$1, C11.P$1, C12.P$1, C18.P$1, C19.P$1, C2.P$1, C20.P$1, C24.P$1, C26.P$1, C29.P$1, C3.P$1, C4.P$1, C5.P$1, C6.P$1, C7.P$1, C8.P$1, R18.P$2, R34.P$1, R35.P$1, R5.P$2, R6.P$2, R7.P$2, R84.P$2, U$5.5
- net 5V: now also C108.P$1, R306.P$1, R307.P$2, U203.5; no longer C9.P$1, R52.P$2, R61.P$1, U13.5
- net GND: now also C101.P$2, C102.P$2, C103.P$2, C104.P$2, C105.P$2, C106.P$2, C107.P$2, C108.P$2, C109.P$2, C110.P$2, C111.P$2, C205.P$2, C206.P$2, C207.P$2, C208.P$2, C209.P$2, C301.P$2, C302.P$2, C402.-, C403.P$2, D206.1, D208.C, J201.GND, J201.GND@1, J201.GND@2, J201.GND@3, J201.GND@4, R208.P$1, R406.P$1, SW101.3, SW101.4, U203.3, U205.2, U205.PAD; no longer C1.P$2, C10.P$2, C11.P$2, C12.P$2, C13.-, C17.P$2, C18.P$2, C19.P$2, C2.P$2, C20.P$2, C21.P$2, C24.P$2, C25.P$2, C26.P$2, C27.P$2, C28.P$2, C29.P$2, C3.P$2, C4.P$2, C5.P$2, C6.P$2, C7.P$2, C8.P$2, C9.P$2, D4.1, D5.P$1, J8.GND, J8.GND@1, J8.GND@2, J8.GND@3, J8.GND@4, R38.P$1, R83.P$1, SW1.3, SW1.4, U$5.2, U$5.PAD, U13.3
- net I2C0-SCL-SENS: now also R102.P$1; no longer R7.P$1
- net I2C0-SDA-SENS: now also R101.P$1; no longer R6.P$1
- net MAIN_HFXTAL_N: now also Y101.1; no longer Y2.1
- net MAIN_HFXTAL_P: now also Y101.2; no longer Y2.2
- net MAIN_LFXTAL_N: now also Y102.4; no longer Y1.4
- net MAIN_LFXTAL_P: now also Y102.1; no longer Y1.1
- net N$13: now also D207.C, U205.13; no longer D3.P$1, U$5.13
- net N$15: now also D209.C, U205.14; no longer D2.P$1, U$5.14
- net N$16: now also D209.A, R210.P$2; no longer D2.P$2, R34.P$2
- net N$17: now also R213.P$1; no longer R1.P$1
- net N$19: now also D207.A, R209.P$2; no longer D3.P$2, R35.P$2
- net N$34: now also R307.P$1; no longer R52.P$1
- net N$35: now also D208.A; no longer D5.P$2
- net N$38: now also R313.1; no longer R47.1
- net N$4: now also R214.P$1; no longer R60.P$1
- net N$40: now also R313.2, R315.1; no longer R47.2, R49.1
- net N$42: now also R315.2; no longer R49.2
- net N$51: now also D301.A, R306.P$2; no longer D7.P$2, R61.P$2
- net N$69: now also U203.1; no longer U13.1
- net N$7: now also D301.C; no longer D7.P$1
- net N$77: now also U203.2; no longer U13.2
- net PRS-CH11-SSR-OUT: now also TP301.1
- net QSPI_CS0: now also R105.P$1; no longer R5.P$1
- net SDIO-CD: now also R106.P$1; no longer R84.P$1
- net U0RX-USB-TX: now also U205.21; no longer U$5.21
- net U0TX-USB-RX: now also U205.20; no longer U$5.20
- net UART_VBUS: now also R207.P$1, R208.P$2, U205.8; no longer R37.P$1, R38.P$2, U$5.8
- net US1-CS-TFT: now also R206.P$1; no longer R18.P$1
- net USB-D+: now also JP202.1; no longer D4.3, J8.VBUS, JP1.1, JP1.2
- net USB-D-: now also JP201.1; no longer D4.2, J8.D+, JP2.1, JP2.2
- net USB-ID: now also J201.ID; no longer J8.ID
- net USB-RST: now also U205.9; no longer U$5.9
- net USB-SUS: now also U205.17; no longer U$5.17
- net USB-UART-D+: now also JP202.3, U205.3; no longer JP1.3, U$5.3
- net USB-UART-D-: now also JP201.3, U205.4; no longer JP2.3, U$5.4
- net V_USB: now also D206.4, J201.VBUS, R207.P$2, TP202.1; no longer C27.P$1, D4.4, J8.D-, R37.P$2, U$5.7
- net WTIM1-CC1-ZERO-CROSS: now also TP302.1, U101.64
Routing:
- net 2.8V: track 0.00 -> 429.0 mm, vias 0 -> 27
- net 5V: track 100.9 -> 312.2 mm, vias 4 -> 12
- net GND: track 0.00 -> 164.4 mm, vias 0 -> 425
- net I2C0-SDA-SENS: track 0.00 -> 84.1 mm, vias 0 -> 2
- net I2C0-SCL-SENS: track 0.00 -> 81.4 mm, vias 0 -> 2
- net WTIM1-CC1-ZERO-CROSS: track 3.19 -> 77.3 mm, vias 0 -> 2
- net 12V: track 60.8 -> 122.3 mm, vias 0 -> 2
- net USB-ID: track 0.00 -> 55.1 mm, vias 0 -> 2
- net PRS-CH11-SSR-OUT: track 0.00 -> 46.9 mm
- net AC-N: track 50.7 -> 97.4 mm
- net TIM5-CC1-FAN0-CTRL: track 0.00 -> 43.8 mm, vias 0 -> 2
- net TIM3-CC0-FAN1-SNSE: track 1.85 -> 42.4 mm, vias 0 -> 2
- net !RESET: track 10.4 -> 50.2 mm, vias 0 -> 4
- net TIM5-CC0-FAN0-GND: track 0.00 -> 38.6 mm, vias 0 -> 2
- net 12V-FB: track 0.00 -> 36.9 mm, vias 0 -> 2
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- added copper zone on layer 16, net AC-L
- added copper zone on layer 1, net GND
- added copper zone on layer 16, net GND
Other:
- board text added: "Revision: hv0a Date: 05-19"
