File: pcb/r3eflow-v3.sch (EAGLE design)
At the start: 107 parts, among them J1 SH-6, J3 2EDG-2P, J4 2EDG-2P, J5 2EDG-2P, J6 2EDG-2P, J7 2EDG-2P, J8 3X1_2.54, J9 2X1_2.54, Q1 BC817-40, Q2 BC817-40, Q3 BC817-40, Q4 BC817-40, U1 EFM32GG11B8XX_Q64, U2 SST26VF064B, U3 MIC39100, U4 MCP9600, U5 ER-TFT035-6BOT, U6 H11AA1, U7 MCP9600, Y1 32.768KHz, Y2 8MHz

Commit message: pcb work
Parts:
- added C29: (no value), Passive Components > Capacitors > Multilayer Ceramic Capacitors MLCC:MLCC0603
- added D5: SML-D12, Opto-electronics > LED Emitters:SML-D12
- added M1: HM-11, Embedded > BLE Module:HM-11
- added R48: (no value), Passive Components > Resistors > Chip Resistors:RESISTOR0603
Connections:
- net RXD renamed USB-RX
- net TXD renamed USB-TX
- new net BLE-!RST: M1.!RST!@11
- new net BLE-KEY: M1.PIO0@16
- new net BLE-RX: M1.RX@4
- new net BLE-TX: M1.TX@2
- new net N$35: D5.AN, R48.P$2
- new net N$36: M1.PIO1@15, R48.P$1
- new net USB-SUS: U$5.SUSPEND@17
- new net USB-WKUP: U$5.GPIO3-WKUP@11
- net 3.3V: now also C29.P$1, M1.VCC@9
- net BTN_1: now also C20.P$2
- net BTN_2: now also C21.P$2
- net BTN_3: now also C22.P$2
- net BTN_4: now also C23.P$2
- net BTN_5: now also C24.P$2
- net GND: now also C29.P$2, D5.CA, M1.GND@12
- net N$12: no longer C23.P$2
- net N$14: no longer C24.P$2
- net N$3: no longer C20.P$2
- net N$6: no longer C21.P$2
- net N$8: no longer C22.P$2
Other:
- note added: "Bluetooth"
- moved on the sheet: R15, R30, R31, R32, R33

Commit message: pcb work
Parts:
- removed J5: 2EDG-2P, Connectors > Other:2EDG-2P
- added C30, C31, C32, C34, C35: 100n, Passive Components > Capacitors > Multilayer Ceramic Capacitors MLCC:MLCC0603
- added C33, C36: 10u, Passive Components > Capacitors > Tantalum Capacitors:CAPACITOR_TAN3216
- added C37, C38: (no value), Passive Components > Capacitors > Multilayer Ceramic Capacitors MLCC:MLCC0603
- added D6, D8: SK54L, Semiconductors > Discrete Semiconductors > Diodes & Rectifiers > Schottky Diodes & Rectifiers:SK54L
- added D7: SML-D12, Opto-electronics > LED Emitters:SML-D12
- added J10, J11: 4P-PC-FAN, Thermal Management > Fans & Blowers:4P-PC-FAN
- added J12, J13: PCC-SMP, Connectors > Other:PCC-SMP
- added J2: 3X1_2.54, Connectors > Header:3X1_2.54
- added KK1: SK104, Thermal Management > Heatsinks:SK104
- added L1, L2: 68uH, Passive Components > Inductors, Chokes & Coils:INDUCTOR1207
- added Q10, Q11, Q12, Q6, Q7, Q8, Q9: BC817-40, Semiconductors > Discrete Semiconductors > Transistors > Bipolar Transistors - BJT:BC817-40
- added Q5: MOC3051, Opto-electronics > Optocouplers\Photocouplers:MOC3051
- added R45, R46, R47, R49: (no value), Passive Components > Resistors > Chip Resistors:RESISTOR_1206
- added R50, R51: 54.9k, Passive Components > Resistors > Chip Resistors:RESISTOR_1206
- added R52, R60, R61, R62, R63, R64, R65, R66, R67, R68, R69, R70, R71, R72, R73, R74, R75, R76, R77, R78, R79, R80, R81, R82, R83, R84, R85: (no value), Passive Components > Resistors > Chip Resistors:RESISTOR0603
- added R53, R59: 1.2k, Passive Components > Resistors > Chip Resistors:RESISTOR0603
- added R54, R55: 10M, Passive Components > Resistors > Chip Resistors:RESISTOR0603
- added R56, R57: 10k, Passive Components > Resistors > Chip Resistors:RESISTOR0603
- added R58: 3.01k, Passive Components > Resistors > Chip Resistors:RESISTOR0603
- added U$7: HLK-PM01, Power > AC\DC Converters:HLK-PM01
- added U$8: BTA16, Semiconductors > Discrete Semiconductors > Thyristors > Triacs:BTA16
- added U8, U9: MIC4682, Power > Switching Controllers:MIC4682
- C15: value 1u -> 100n
- C16: value 1u -> 10u; device Passive Components > Capacitors > Multilayer Ceramic Capacitors MLCC:MLCC0603 -> Passive Components > Capacitors > Tantalum Capacitors:CAPACITOR_TAN3216
- C17: value (none) -> 100n
- C9: value (none) -> 10u; device Passive Components > Capacitors > Multilayer Ceramic Capacitors MLCC:MLCC0603 -> Passive Components > Capacitors > Tantalum Capacitors:CAPACITOR_TAN3216
- J4: value 2EDG-2P -> MICROSD; device Connectors > Other:2EDG-2P -> Connectors > card socket:MICROSD
- J7: value 2EDG-2P -> 3X1_2.54; device Connectors > Other:2EDG-2P -> Connectors > Header:3X1_2.54
- R36: value (none) -> 3.01k
- R40, R41: value (none) -> 54.9k; device Passive Components > Resistors > Chip Resistors:RESISTOR0603 -> Passive Components > Resistors > Chip Resistors:RESISTOR_1206
- R42: value (none) -> 10k
Connections:
- removed net SERVO-SIG: J8-1.S
- new net 12V: C13.P$1, C14.AN, C30.P$1, C34.P$1, F1.1, J10-12VDC.S, J11-12VDC.S, R1.P$2, R54.P$2, R55.P$2, R60.P$2, R71.P$2, R73.P$2, R82.P$2, U8.IN, U9.IN
- new net 12V-FB: C25.P$1, R82.P$1, R83.P$2
- new net 2.8V: C1.P$1, C12.P$1, C16.AN, C18.P$1, C19.P$1, C2.P$1, C26.P$1, C29.P$1, C3.P$1, C32.P$1, C4.P$1, C5.P$1, C6.P$1, J1-1.S, J4.4, M1.VCC@9, R10.P$2, R11.P$2, R12.P$2, R13.P$2, R14.P$2, R18.P$2, R22.P$2, R28.P$2, R34.P$1, R35.P$1, R42.P$2, R44.P$2, R5.P$2, R6.P$2, R7.P$2, R8.P$2, R84.P$2, R85.P$2, R9.P$2, U$5.VIO@5, U1.AVDD, U1.DVDD, U1.IOVDD0@0, U1.IOVDD0@1, U1.IOVDD0@2, U1.VREGVDD, U2.VCC, U3.VOUT, U4.VDD@8, U5.!RD, U5.IM0, U5.IM1, U5.IM2, U5.VCI, U5.VDDI@0, U5.VDDI@1, U7.ADDR@16, U7.VDD@8
- new net 3.6V: C15.P$1, C31.P$1, C33.AN, L1.P$2, R36.P$2, R78.P$2, U3.VIN
- new net 3.6V-FB: C38.P$1, R78.P$1, R79.P$2
- new net 5V-FB: C37.P$1, R80.P$1, R81.P$2
- new net AC-L: J3-2.S, J6-1.S, R40.P$1, U$7.AC2
- new net AC-N: J3-1.S, R50.P$1, U$7.AC1, U$8.A1
- new net FAN0-CTRL: R70.P$1
- new net FAN0-GND: R68.P$1
- new net FAN0-SNSE: R74.P$1, R75.P$2
- new net FAN1-CTRL: R72.P$1
- new net FAN1-GND: R69.P$1
- new net FAN1-SNSE: R76.P$1, R77.P$2
- new net N$34: Q5.AN, R52.P$1
- new net N$37: Q5.MAIN@1, R45.P$1
- new net N$38: Q5.MAIN@2, R47.P$1
- new net N$39: R45.P$2, R46.P$1
- new net N$40: R47.P$2, R49.P$1
- new net N$41: J6-2.S, R46.P$2, U$8.A2
- new net N$42: R49.P$2, U$8.G
- new net N$43: R36.P$1, R53.P$2, U9.FB
- new net N$44: R54.P$1, R57.P$2, U9.ISET
- new net N$45: D6.C, L2.P$1, U8.SW
- new net N$46: R58.P$1, R59.P$2, U8.FB
- new net N$47: R55.P$1, R56.P$2, U8.ISET
- new net N$48: C28.P$1, U$5.VDD@6
- new net N$49: Q6.BA1, R62.P$2
- new net N$50: J2-1.S, Q6.C03, R63.P$1
- new net N$51: D7.AN, R61.P$2
- new net N$52: J7-1.S, Q7.C03, R65.P$1
- new net N$53: Q7.BA1, R64.P$2
- new net N$54: Q8.BA1, R66.P$2
- new net N$55: J8-1.S, Q8.C03, R67.P$1
- new net N$56: Q9.BA1, R68.P$2
- new net N$57: J11-GND.S, Q9.C03
- new net N$58: Q10.BA1, R70.P$2
- new net N$59: J11-CTRL.S, Q10.C03, R71.P$1
- new net N$60: Q11.BA1, R69.P$2
- new net N$61: Q12.BA1, R72.P$2
- new net N$62: J10-CTRL.S, Q12.C03, R73.P$1
- new net N$63: J10-GND.S, Q11.C03
- new net N$64: J11-SENSE.S, R74.P$2
- new net N$65: J10-SENSE.S, R76.P$2
- new net N$67: J4.2, R85.P$1
- new net SD-CD: J4.CD@9, R84.P$1
- new net SERVO0-SIG: R62.P$1
- new net SERVO1-SIG: R66.P$1
- new net SERVO2-SIG: R64.P$1
- new net USB-RST: U$5.RSTB@9
- new net V_USB: C27.P$1, D4.4, R37.P$2, U$5.VREGIN@7, U$6.VBUS
- net !RESET: now also J1-2.S; no longer J12.S
- net 3.3V: no longer C1.P$1, C12.P$1, C16.P$1, C17.P$1, C18.P$1, C19.P$1, C2.P$1, C25.P$1, C26.P$1, C27.P$1, C28.P$1, C29.P$1, C3.P$1, C4.P$1, C5.P$1, C6.P$1, J11.S, M1.VCC@9, R10.P$2, R11.P$2, R12.P$2, R13.P$2, R14.P$2, R18.P$2, R22.P$2, R28.P$2, R34.P$1, R35.P$1, R36.P$1, R42.P$2, R44.P$2, R5.P$2, R6.P$2, R7.P$2, R8.P$2, R9.P$2, U$5.VDD@6, U$5.VIO@5, U$5.VREGIN@7, U1.AVDD, U1.DVDD, U1.IOVDD0@0, U1.IOVDD0@1, U1.IOVDD0@2, U1.VREGVDD, U2.VCC, U3.VOUT, U4.VDD@8, U5.!RD, U5.IM0, U5.IM1, U5.IM2, U5.LEDA, U5.VCI, U5.VDDI@0, U5.VDDI@1, U7.ADDR@16, U7.VDD@8
- net 5V: now also C35.P$1, C36.AN, J2-2.S, J7-2.S, L2.P$2, R52.P$2, R58.P$2, R61.P$1, R63.P$2, R65.P$2, R67.P$2, R80.P$2, U5.LEDA; no longer B1.A, C13.P$1, C14.AN, C15.P$1, F1.1, J6-1.S, R1.P$2, U3.VIN
- net GND: now also C16.CA, C30.P$2, C31.P$2, C32.P$2, C33.CA, C34.P$2, C35.P$2, C36.CA, C37.P$2, C38.P$2, C9.CA, D6.A, D8.A, J1-6.S, J1-CASE.S, J12-BAR.S, J13-BAR.S, J2-3.S, J4.6, J4.BODY@10, J7-3.S, Q10.EM2, Q11.EM2, Q12.EM2, Q6.EM2, Q7.EM2, Q8.EM2, Q9.EM2, R53.P$1, R56.P$1, R57.P$1, R59.P$1, R75.P$1, R77.P$1, R79.P$1, R81.P$1, R83.P$1, U$7.-VO, U8.GND@1, U8.GND@2, U8.GND@3, U8.SHDN, U9.GND@1, U9.GND@2, U9.GND@3, U9.SHDN; no longer C16.P$2, C9.P$2, J16.S, J1CASE.S, J3-2.S
- net N$20: now also R40.P$2, R41.P$1; no longer J7-1.S, R40.P$1
- net N$21: now also R41.P$2; no longer R40.P$2
- net N$28: now also D8.C, L1.P$1, U9.SW; no longer R36.P$2, U$5.RSTB@9
- net N$29: now also R51.P$2; no longer R41.P$2
- net N$30: now also R50.P$2, R51.P$1; no longer J7-2.S, R41.P$1
- net N$31: now also U$7.+VO; no longer J3-1.S
- net N$4: now also B1.A, R60.P$1; no longer D4.4, R37.P$2, U$6.VBUS
- net N$7: now also D7.CA, Q5.CA; no longer J6-2.S
- net N$9: now also C17.P$1, C9.AN; no longer C9.P$1
- net SWCLK: now also J1-3.S; no longer J13.S
- net SWDIO: now also J1-4.S; no longer J14.S
- net SWO: now also J1-5.S; no longer J15.S
- net TC_VIN0+: now also J12-T+.S; no longer J4-1.S
- net TC_VIN0-: now also J12-T-.S; no longer J4-2.S
- net TC_VIN1+: now also J13-T+.S; no longer J5-1.S
- net TC_VIN1-: now also J13-T-.S; no longer J5-2.S
Other:
- note added: "Io(max) ~ 2A DS pag. 5"
- note added: "Vo = 1.23 * (R3/R4 + 1) Vo ~ 4.31V"
- note removed: "Decouple"
- note removed: "SPI Flash Decouple"
- moved on the sheet: B1, B2, B3, B4, B5, B6, C1, C10, C11, C12, C13, C14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

Commit message: pn532 dev
Parts:
- removed C15, C32: 100n, Passive Components > Capacitors > Multilayer Ceramic Capacitors MLCC:MLCC0603
- removed U3: MIC39100, Power > LDO Voltage Regulators:MIC39100
Connections:
- net 2.8V: now also U1.VREGO; no longer C32.P$1, U3.VOUT
- net 3.6V: no longer C15.P$1, U3.VIN
- net 5V: now also U1.VREGI
- net GND: no longer C15.P$2, C32.P$2, U3.GND_(TAB), U3.GND_(TAB)_2
Other:
- moved on the sheet: C1, C2, C3, C4, C5, C6

Commit message: pcb work
Parts:
- removed B2, B3, B4, B5, B6: PUSH-SILENT, Eletromechanical > Switches > Tactile Switches:PUSH-SILENT
- removed C30, C31: 100n, Passive Components > Capacitors > Multilayer Ceramic Capacitors MLCC:MLCC0603
- removed C33, C36: 10u, Passive Components > Capacitors > Tantalum Capacitors:CAPACITOR_TAN3216
- removed C37, C38: (no value), Passive Components > Capacitors > Multilayer Ceramic Capacitors MLCC:MLCC0603
- removed D1: WS2812B, Opto-electronics > LED Emitters:WS2812B
- removed J8: 3X1_2.54, Connectors > Header:3X1_2.54
- removed J9: 2X1_2.54, Connectors > Header:2X1_2.54
- removed Q2, Q8: BC817-40, Semiconductors > Discrete Semiconductors > Transistors > Bipolar Transistors - BJT:BC817-40
- removed R12, R13, R19, R20, R21, R22, R23, R25, R26, R27, R28, R29, R3, R30, R31, R32, R33, R4, R43, R44, R66, R67, R78, R79, R80, R81, R85: (no value), Passive Components > Resistors > Chip Resistors:RESISTOR0603
- removed R36: 3.01k, Passive Components > Resistors > Chip Resistors:RESISTOR0603
- removed R53: 1.2k, Passive Components > Resistors > Chip Resistors:RESISTOR0603
- removed R54: 10M, Passive Components > Resistors > Chip Resistors:RESISTOR0603
- removed R57: 10k, Passive Components > Resistors > Chip Resistors:RESISTOR0603
- removed U9: MIC4682, Power > Switching Controllers:MIC4682
- added C15: 100n, Passive Components > Capacitors > Multilayer Ceramic Capacitors MLCC:MLCC0603
- added C32: (no value), Passive Components > Capacitors > Multilayer Ceramic Capacitors MLCC:MLCC0603
- added D10, D11, D12, D9: WS2812B, Opto-electronics > LED Emitters:WS2812B3535
- added J5: 2X1_2.54, Connectors > Header:2X1_2.54
- added U11: 74HC123, Semiconductors > Integrated Circuits - ICs > Logic ICs > Logic Gates:74HC123
- added U12: 74LVC1G08, Semiconductors > Integrated Circuits - ICs > Logic ICs > Logic Gates:74LVC1G08
- added U13: 74LVC1G32, Semiconductors > Integrated Circuits - ICs > Logic ICs > Logic Gates:74LVC1G32
- C1, C18, C2, C20, C3, C4, C5, C6, C7: value (none) -> 100n
- C13: value 100n -> (none); device Passive Components > Capacitors > Multilayer Ceramic Capacitors MLCC:MLCC0603 -> Passive Components > Capacitors > Aluminium Electrolytic Capacitors:CAPACITOR_ELD
- C14: device Passive Components > Capacitors > Aluminium Electrolytic Capacitors:CAPACITOR_EL10X10 -> Passive Components > Capacitors > Aluminium Electrolytic Capacitors:CAPACITOR_ELD
- C16: value 10u -> (none); device Passive Components > Capacitors > Tantalum Capacitors:CAPACITOR_TAN3216 -> Passive Components > Capacitors > Multilayer Ceramic Capacitors MLCC:MLCC0603
- C17: value 100n -> 1u
- C21: value (none) -> 4u7
- C22, C23: value (none) -> 100p
- C24: value (none) -> 1u
- C35: value 100n -> (none)
- C9: value 10u -> 1u; device Passive Components > Capacitors > Tantalum Capacitors:CAPACITOR_TAN3216 -> Passive Components > Capacitors > Multilayer Ceramic Capacitors MLCC:MLCC0603
- D8: value SK54L -> WS2812B; device Semiconductors > Discrete Semiconductors > Diodes & Rectifiers > Schottky Diodes & Rectifiers:SK54L -> Opto-electronics > LED Emitters:WS2812B3535
- L1: value 68uH -> 4.7nH; device Passive Components > Inductors, Chokes & Coils:INDUCTOR1207 -> Passive Components > Inductors, Chokes & Coils:INDUCTOR0805
- R14, R15: value (none) -> 3k95
- R59: value 1.2k -> 1k
- U1: value EFM32GG11B8XX_Q64 -> EFM32GG11B8XX_Q100; device Semiconductors > Embedded Processors & Controllers > Microcontrollers - MCU:EFM32GG11B8XX_Q64 -> Semiconductors > Embedded Processors & Controllers > Microcontrollers - MCU:EFM32GG11B8XX_Q100
Connections:
- removed net 3.6V: C31.P$1, C33.AN, L1.P$2, R36.P$2, R78.P$2
- removed net 3.6V-FB: C38.P$1, R78.P$1, R79.P$2
- removed net 5V-FB: C37.P$1, R80.P$1, R81.P$2
- removed net BLE-RX: M1.RX@4
- removed net BLE-TX: M1.TX@2
- removed net BTN_1: C20.P$2, R30.P$2
- removed net BTN_2: C21.P$2, R15.P$2
- removed net BTN_3: C22.P$2, R31.P$2
- removed net BTN_4: C23.P$2, R32.P$2
- removed net BTN_5: C24.P$2, R33.P$2
- removed net DOOR-SWITCH: R43.P$2
- removed net LED_DI: R4.P$1
- removed net N$11: D1.DI, Q2.C03, R3.P$1
- removed net N$27: R20.P$2, U4.VIN-@4
- removed net N$28: D8.C, L1.P$1, U9.SW
- removed net N$3: B2.3, R10.P$1, R30.P$1
- removed net N$32: J9-2.S
- removed net N$33: J9-1.S, R43.P$1, R44.P$1
- removed net N$43: R36.P$1, R53.P$2, U9.FB
- removed net N$44: R54.P$1, R57.P$2, U9.ISET
- removed net N$54: Q8.BA1, R66.P$2
- removed net N$55: J8-1.S, Q8.C03, R67.P$1
- removed net N$67: J4.2, R85.P$1
- removed net SD-CD: J4.CD@9, R84.P$1
- removed net SERVO1-SIG: R66.P$1
- removed net US1-MISO-TFT: U5.SDO
- removed net US1-MOSI-TFT: U5.SDA
- removed net USB-WKUP: U$5.GPIO3-WKUP@11
- removed net ZERO-CROSS: R42.P$1, U6.C
- new net !LED_CS: U11.A.!A, U11.B.!A
- new net DOOR-SW: C16.P$1, R11.P$2
- new net LED_MOSI: U12.A.A
- new net LED_SCK: U11.B.B, U12.A.B
- new net N$69: U11.B.Q, U13.A.B
- new net N$77: U11.A.Q, U13.A.A
- new net N$78: U11.A.B, U12.A.Y
- new net N$79: C22.P$2, R14.P$2, U11.A.R/C
- new net N$80: C22.P$1, U11.A.C
- new net N$81: C23.P$2, R15.P$2, U11.B.R/C
- new net N$82: C23.P$1, U11.B.C
- new net SDIO-CD: J4.CD@9, R84.P$1, U1.PF8
- new net SDIO-CLK: J4.5, U1.PE13
- new net SDIO-CMD: J4.3, U1.PE12
- new net SDIO-DAT0: J4.7, U1.PE11
- new net SDIO-DAT1: J4.8, U1.PE10
- new net SDIO-DAT2: J4.1, U1.PE9
- new net SDIO-DAT3: J4.2, U1.PE8
- new net U1RX-BLE-TX: M1.TX@2, U1.PE3
- new net U1TX-BLE-RX: M1.RX@4, U1.PE2
- new net US0-MISO-TFT: U1.PC1, U5.SDO
- new net US0-MOSI-TFT: U1.PC0, U5.SDA
- new net WTIM1-CC1-ZERO-CROSS: R42.P$1, U1.PE4, U6.C
- net 12V: now also C13.AN; no longer C13.P$1, C14.AN, C30.P$1, R54.P$2, U9.IN
- net 12V-FB: now also U1.PD0
- net 2.8V: now also C10.P$1, C11.P$1, C20.P$1, C24.P$1, C7.P$1, C8.P$1, U1.IOVDD0@3, U1.IOVDD0@4; no longer C16.AN, R11.P$2, R12.P$2, R13.P$2, R14.P$2, R22.P$2, R28.P$2, R44.P$2, R85.P$2, U1.DVDD
- net 3.3V: now also U12.PW.VCC; no longer C10.P$1, C11.P$1, C8.P$1
- net 5V: now also C14.AN, C15.P$1, C32.P$1, C9.P$1, D10.VDD, D11.VDD, D12.VDD, D8.VDD, D9.VDD, R14.P$1, R15.P$1, U1.VBUS, U11.A.!RD, U11.B.!RD, U11.PW.VCC, U13.PW.VCC; no longer C36.AN, C7.P$1, D1.VDD, J8-2.S, R3.P$2, R67.P$2, R80.P$2
- net GND: now also C13.CA, C15.P$2, C16.P$2, C20.P$2, C21.P$2, C24.P$2, C32.P$2, C9.P$2, D10.VSS, D11.VSS, D12.VSS, D8.VSS, D9.VSS, J5-2.S, U1.VSS@3, U11.PW.GND, U12.PW.GND, U13.PW.GND; no longer B2.1, B3.1, B4.1, B5.1, B6.1, C13.P$2, C16.CA, C20.P$1, C21.P$1, C22.P$1, C23.P$1, C24.P$1, C30.P$2, C31.P$2, C33.CA, C36.CA, C37.P$2, C38.P$2, C9.CA, D1.VSS, D8.A, J8-3.S, Q2.EM2, Q8.EM2, R21.P$1, R23.P$1, R27.P$1, R29.P$1, R53.P$1, R57.P$1, R79.P$1, R81.P$1, U9.GND@1, U9.GND@2, U9.GND@3, U9.SHDN
- net I2C0-SCL-SENS: now also U1.PD7
- net I2C0-SDA-SENS: now also U1.PD6
- net I2C1-SCL-TFT: now also U1.PC5
- net I2C1-SDA-TFT: now also U1.PC4
- net MAIN_HFXTAL_N: now also U1.PB14
- net MAIN_HFXTAL_P: now also U1.PB13
- net MAIN_LFXTAL_N: now also U1.PB8
- net MAIN_LFXTAL_P: now also U1.PB7
- net N$1: now also J5-1.S, R10.P$1, R11.P$1; no longer R25.P$2, U7.VIN+@2
- net N$10: now also D10.DI, D9.DO; no longer Q2.BA1, R4.P$2
- net N$12: now also D8.DI, U13.A.Y; no longer B5.3, R13.P$1, R32.P$1
- net N$14: now also L1.P$2, U1.VREGSW; no longer B6.3, R14.P$1, R33.P$1
- net N$2: now also D8.DO, D9.DI; no longer R26.P$2, U7.VIN-@4
- net N$26: now also C21.P$1, L1.P$1, U1.DVDD; no longer R19.P$2, U4.VIN+@2
- net N$6: now also D10.DO, D11.DI; no longer B3.3, R11.P$1, R15.P$1
- net N$8: now also D11.DO, D12.DI; no longer B4.3, R12.P$1, R31.P$1
- net N$9: no longer C9.AN
- net QSPI_CLK: now also U1.PF6
- net QSPI_CS0: now also U1.PF7
- net QSPI_D0: now also U1.PD9
- net QSPI_D1: now also U1.PD10
- net QSPI_D2: now also U1.PD11
- net QSPI_D3: now also U1.PD12
- net TC_VIN0+: now also U4.VIN+@2; no longer R19.P$1, R21.P$2, R22.P$1
- net TC_VIN0-: now also U4.VIN-@4; no longer R20.P$1, R23.P$2
- net TC_VIN1+: now also U7.VIN+@2; no longer R25.P$1, R27.P$2, R28.P$1
- net TC_VIN1-: now also U7.VIN-@4; no longer R26.P$1, R29.P$2
- net USB-RX: now also U1.PA3
- net USB-TX: now also U1.PA4
Other:
- note added: "Vo = 1.23 * (R1/R2 + 1) Vo ~ 4.93V"
- note added: "long pulser (1)"
- note added: "short pulser (0)"
- note removed: "Buttons"
- note removed: "Vo = 1.23 * (R3/R4 + 1) Vo ~ 4.31V"
- moved on the sheet: B1, C1, C10, C11, C14, C2, C22, C23, C25, C29, C3, C34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

Commit message: sync
Parts:
- removed U$6: USB-SHIELD, Connectors > USB:USB-SHIELD
- added J8: USB-SHIELD, Connectors > USB:USB-SHIELD
- added JP1, JP2: JUMPER-SMT_3_1-NC_PASTE_SILK, Utility > Board:JUMPER-SMT_3_1-NC_PASTE_SILK
Connections:
- net I2C1-SCL-TFT renamed I2C1-SCL-TTFT
- net I2C1-SDA-TFT renamed I2C1-SDA-TTFT
- net USB-RX renamed U0TX-USB-RX
- net USB-TX renamed U0RX-USB-TX
- removed net !LED_CS: U11.A.!A, U11.B.!A
- removed net !TFT-IRQ: U5.X-/!IRQ!
- removed net !TFT-RST: U5.Y-/!RST!
- removed net FAN0-CTRL: R70.P$1
- removed net FAN0-GND: R68.P$1
- removed net FAN0-SNSE: R74.P$1, R75.P$2
- removed net FAN1-CTRL: R72.P$1
- removed net FAN1-GND: R69.P$1
- removed net FAN1-SNSE: R76.P$1, R77.P$2
- removed net LED_MOSI: U12.A.A
- removed net LED_SCK: U11.B.B, U12.A.B
- removed net SERVO0-SIG: R62.P$1
- removed net SERVO2-SIG: R64.P$1
- removed net SSR-OUT: R39.P$1
- removed net TIM3_CC2_BUZZ: R2.P$1
- removed net UART-D+: D4.3, U$5.D+@3, U$6.D+
- removed net UART-D-: D4.2, U$5.D-@4, U$6.D-
- removed net US0-MISO-TFT: U1.PC1, U5.SDO
- removed net US0-MOSI-TFT: U1.PC0, U5.SDA
- removed net WTIM2_CC1_TFT_BL: R24.P$1
- new net !LED-CS: U1.PE6, U11.1.!A, U11.2.!A
- new net !TTFT-IRQ: U1.PB3, U5.X-/!IRQ!
- new net !TTFT-RST: U1.PB6, U5.Y-/!RST!
- new net PRS-CH11-SSR-OUT: R39.P$1, U1.PD5
- new net TIM0-CC0-BUZZ: R2.P$1, U1.PA8
- new net TIM1-CC0-TFT-BL: R24.P$1, U1.PB0
- new net TIM2-CC2FAN0-SNSE: R74.P$1, R75.P$2, U1.PC10
- new net TIM3-CC0-FAN1-SNSE: R76.P$1, R77.P$2, U1.PA6
- new net TIM5-CC0-FAN0-GND: R68.P$1, U1.PC8
- new net TIM5-CC1-FAN0-CTRL: R70.P$1, U1.PC9
- new net TIM6-CC0-FAN1-GND: R69.P$1, U1.PD1
- new net TIM6-CC1-FAN1-CTRL: R72.P$1, U1.PD2
- new net US0-LED-MOSI: U1.PE7, U12.1.A
- new net US0-LED-SCK: U1.PE5, U11.2.B, U12.1.B
- new net US1-MISO-TFT: U1.PC2, U5.SDO
- new net US1-MOSI-TFT: U1.PC1, U5.SDA
- new net USB-D+: D4.3, J8.VBUS, JP1.1, JP1.2, U1.PF11
- new net USB-D-: D4.2, J8.D+, JP2.1, JP2.2, U1.PF10
- new net USB-ID: J8._ID, U1.PF12
- new net USB-UART-D+: JP1.3, U$5.D+@3
- new net USB-UART-D-: JP2.3, U$5.D-@4
- new net WTIM0-CC0-ZERO-CROSS: U1.PE4
- new net WTIM2-CC0-SERVO0-SIG: R62.P$1, U1.PD3
- new net WTIM2-CC1-SERVO1-SIG: R64.P$1, U1.PD4
- net !RESET: now also J1.2.S; no longer J1-2.S
- net !TFT_RESET: now also U1.PB5
- net 2.8V: now also J1.1.S; no longer J1-1.S
- net 5V: now also U11.1.!RD, U11.2.!RD; no longer U11.A.!RD, U11.B.!RD
- net AC-L: now also J3.2.S, J6.1.S; no longer J3-2.S, J6-1.S
- net AC-N: now also J3.1.S; no longer J3-1.S
- net BLE-!RST: now also U1.PD8
- net BLE-KEY: now also U1.PE1
- net DOOR-SW: now also U1.PC7
- net GND: now also J1.6.S, J1.TAB.S, J12.BAR.S, J13.BAR.S, J8.CASE, J8.GND; no longer J1-6.S, J1-CASE.S, J12-BAR.S, J13-BAR.S, U$6.GND, U$6.GND@1, U$6.GND@2, U$6.GND@3, U$6.GND@4
- net N$12: now also U13.1.Y; no longer U13.A.Y
- net N$41: now also J6.2.S; no longer J6-2.S
- net N$69: now also U11.2.Q, U13.1.B; no longer U11.B.Q, U13.A.B
- net N$77: now also U11.1.Q, U13.1.A; no longer U11.A.Q, U13.A.A
- net N$78: now also U11.1.B, U12.1.Y; no longer U11.A.B, U12.A.Y
- net N$79: now also U11.1.R/C; no longer U11.A.R/C
- net N$80: now also U11.1.C; no longer U11.A.C
- net N$81: now also U11.2.R/C; no longer U11.B.R/C
- net N$82: now also U11.2.C; no longer U11.B.C
- net SWCLK: now also J1.3.S; no longer J1-3.S
- net SWDIO: now also J1.4.S; no longer J1-4.S
- net SWO: now also J1.5.S; no longer J1-5.S
- net TC_VIN0+: now also J12.T+.S; no longer J12-T+.S
- net TC_VIN0-: now also J12.T-.S; no longer J12-T-.S
- net TC_VIN1+: now also J13.T+.S; no longer J13-T+.S
- net TC_VIN1-: now also J13.T-.S; no longer J13-T-.S
- net TFT-DC: now also U1.PA7
- net US1-CLK-TFT: now also U1.PC3
- net US1-CS-TFT: now also U1.PC0
- net USB-RST: now also U1.PA2
- net USB-SUS: now also U1.PA1
- net V_USB: now also J8.D-; no longer U$6.VBUS
- net WTIM1-CC1-ZERO-CROSS: no longer U1.PE4
Other:
- note added: "verify"
- moved on the sheet: C1, C17, C2, C21, C24, C26, C27, C28, C29, C3, C4, C5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
