File: pcb/r3eflow-v3.sch (EAGLE design)
At the start: 143 parts, among them J1 SH-6, J10 4P-PC-FAN, J11 4P-PC-FAN, J12 PCC-SMP, J13 PCC-SMP, J2 3X1_2.54, J3 2EDG-2P, J4 MICROSD, J5 2X1_2.54, J6 2EDG-2P, J7 3X1_2.54, J8 USB-SHIELD, M1 HM-11, Q1 BC817-40, Q10 BC817-40, Q11 BC817-40, Q12 BC817-40, Q3 BC817-40, Q4 BC817-40, Q5 MOC3051, Q6 BC817-40, Q7 BC817-40, Q9 BC817-40, U1 EFM32GG11B8XX_Q100, U11 74HC123, U12 74LVC1G08, U13 74LVC1G32, U2 SST26VF064B, U4 MCP9600, U5 ER-TFT035-6BOT, U6 H11AA1, U7 MCP9600, U8 MIC4682, Y1 32.768KHz, Y2 8MHz

Commit message: pcb work
Parts:
- removed C10, C11, C26, C27, C28, C29, C32, C35, C8: (no value), Passive Components > Capacitors > Multilayer Ceramic Capacitors MLCC:MLCC0603
- removed C20, C6: 100n, Passive Components > Capacitors > Multilayer Ceramic Capacitors MLCC:MLCC0603
- removed C22, C23: 100p, Passive Components > Capacitors > Multilayer Ceramic Capacitors MLCC:MLCC0603
- removed D10, D11, D12, D8, D9: WS2812B, Opto-electronics > LED Emitters:WS2812B3535
- removed D2, D3, D5, D7: SML-D12, Opto-electronics > LED Emitters:SML-D12
- removed D4: SP0503BAHT, Circuit Protection > ESD Suppressors \ TVS Diodes:SP0503BAHT
- removed J8: USB-SHIELD, Connectors > USB:USB-SHIELD
- removed JP1: JUMPER-SMT_3_1-NC_PASTE_SILK, Utility > Board:JUMPER-SMT_3_1-NC_PASTE_SILK
- removed L1: 4.7nH, Passive Components > Inductors, Chokes & Coils:INDUCTOR0805
- removed M1: HM-11, Embedded > BLE Module:HM-11
- removed Q3: BC817-40, Semiconductors > Discrete Semiconductors > Transistors > Bipolar Transistors - BJT:BC817-40
- removed R14, R15: 3k95, Passive Components > Resistors > Chip Resistors:RESISTOR0603
- removed R16, R17, R18, R24, R34, R35, R48: (no value), Passive Components > Resistors > Chip Resistors:RESISTOR0603
- removed R37: 22.1k, Passive Components > Resistors > Chip Resistors:RESISTOR0603
- removed R38: 47.5k, Passive Components > Resistors > Chip Resistors:RESISTOR0603
- removed U$5: CP2102N, Semiconductors > Integrated Circuits - ICs > Interface ICs > USB Interface IC:CP2102N
- removed U11: 74HC123, Semiconductors > Integrated Circuits - ICs > Logic ICs > Logic Gates:74HC123
- removed U12: 74LVC1G08, Semiconductors > Integrated Circuits - ICs > Logic ICs > Logic Gates:74LVC1G08
- removed U13: 74LVC1G32, Semiconductors > Integrated Circuits - ICs > Logic ICs > Logic Gates:74LVC1G32
- removed U5: ER-TFT035-6BOT, Opto-electronics > Displays:ER-TFT035-6BOT
- added C201, C202: 100p, Passive Components > Capacitors > Multilayer Ceramic Capacitors MLCC:MLCC0603
- added C203, C204, C205, C206, C207, C208, C209: (no value), Passive Components > Capacitors > Multilayer Ceramic Capacitors MLCC:MLCC0603
- added D201, D202, D203, D204, D205: WS2812B, Opto-electronics > LED Emitters:WS2812B3535
- added D206: SP0503BAHT, Circuit Protection > ESD Suppressors \ TVS Diodes:SP0503BAHT
- added D207, D208, D209, D301: LED0603, Opto-electronics > LED Emitters:LED0603
- added J201: USB-SHIELD, Connectors > USB:USB-SHIELD
- added JP202: JUMPER-SMT_3_1-NC_PASTE_SILK, Utility > Board:JUMPER-SMT_3_1-NC_PASTE_SILK
- added L101: 4.7nH, Passive Components > Inductors, Chokes & Coils:INDUCTOR
- added LOGO101: DESIGNEDINPT, Utility > Silkscreen:DESIGNEDINPT
- added LOGO102: RAFAEL_SILVA, Utility > Silkscreen:RAFAEL_SILVA
- added LOGO103: OSHW-LOGOL, Utility > Silkscreen:OSHW-LOGOL
- added M201: HM-11, Embedded > BLE Module:HM-11
- added Q201: BC817-40, Semiconductors > Discrete Semiconductors > Transistors > Bipolar Transistors - BJT:BC817-40
- added R201, R202: 3k95, Passive Components > Resistors > Chip Resistors:RESISTOR0603
- added R203, R204, R205, R206, R209, R210, R211: (no value), Passive Components > Resistors > Chip Resistors:RESISTOR0603
- added R207: 22.1k, Passive Components > Resistors > Chip Resistors:RESISTOR0603
- added R208: 47.5k, Passive Components > Resistors > Chip Resistors:RESISTOR0603
- added TP1, TP10, TP11, TP12, TP13, TP14, TP15, TP16, TP17, TP18, TP19, TP2, TP20, TP201, TP202, TP21, TP22, TP26, TP3, TP301, TP302, TP4, TP5, TP6, TP7, TP8, TP9: TEST_POINT, Utility > Board:TEST_POINT
- added U201: 74LVC1G08, Semiconductors > Integrated Circuits - ICs > Logic ICs > Logic Gates:74LVC1G08
- added U202: 74HC123, Semiconductors > Integrated Circuits - ICs > Logic ICs > Logic Gates:74HC123
- added U203: 74LVC1G32, Semiconductors > Integrated Circuits - ICs > Logic ICs > Logic Gates:74LVC1G32
- added U204: ER-TFT035-6BOT, Opto-electronics > Displays:ER-TFT035-6BOT
- added U205: CP2102N, Semiconductors > Integrated Circuits - ICs > Interface ICs > USB Interface IC:CP2102N
- renumbered B1 to B201, C1 to C104, C12 to C301, C13 to C402, C14 to C404, C15 to C405, C16 to C303, C17 to C109, C18 to C110, C19 to C302, C2 to C105, C21 to C107, C24 to C106, C25 to C403, C3 to C103, C34 to C401, C4 to C102, C5 to C101, C7 to C111, C9 to C108, D6 to D401, F1 to F401, J1 to J102, J10 to J308, J11 to J306, J12 to J301, J13 to J304, J2 to J302, J3 to J401, J4 to J101, J5 to J307, J6 to J305, J7 to J303, JP2 to JP201, KK1 to KK301, L2 to L401, Q1 to Q202, Q10 to Q305, Q11 to Q308, Q12 to Q307, Q4 to Q303, Q5 to Q304, Q6 to Q301, Q7 to Q302, Q9 to Q306, R1 to R213, R10 to R326, R11 to R323, R2 to R212, R39 to R305, R40 to R308, R41 to R310, R42 to R316, R45 to R312, R46 to R314, R47 to R313, R49 to R315, R5 to R105, R50 to R309, R51 to R311, R52 to R307, R55 to R401, R56 to R402, R58 to R403, R59 to R404, R6 to R101, R60 to R214, R61 to R306, R62 to R301, R63 to R302, R64 to R303, R65 to R304, R68 to R319, R69 to R325, R7 to R102, R70 to R318, R71 to R321, R72 to R324, R73 to R328, R74 to R320, R75 to R317, R76 to R327, R77 to R322, R8 to R103, R82 to R405, R83 to R406, R84 to R106, R9 to R104, SW1 to SW101, U$7 to ACDC401, U$8 to D302, U1 to U101, U2 to U102, U4 to U301, U6 to U303, U7 to U302, U8 to U401, Y1 to Y102, Y2 to Y101
Connections:
- net N$46 renamed 5V-FB
- net N$9 renamed DECOUPLE
- net TC0-ALRT2 renamed U4-ALRT2
- net TC0-ALRT3 renamed U4-ALRT3
- net TC0-ALRT4 renamed U4-ALRT4
- net TC1-ALRT2 renamed U7-ALRT2
- net TC1-ALRT3 renamed U7-ALRT3
- net TC1-ALRT4 renamed U7-ALRT4
- removed net 3.3V: U12.PW.VCC
- removed net N$10: D10.DI, D9.DO
- removed net N$12: D8.DI, U13.1.Y
- removed net N$14: L1.P$2, U101.VREGSW
- removed net N$2 (its old number): D8.DO, D9.DI
- removed net N$22: R16.P$2, U5.LEDK@0
- removed net N$23: R17.P$2, U5.LEDK@1
- removed net N$24: Q3.C03, R16.P$1, R17.P$1
- removed net N$26: C107.P$1, L1.P$1, U101.DVDD
- removed net N$48: C28.P$1, U$5.VDD@6
- removed net N$6: D10.DO, D11.DI
- removed net N$79: C22.P$2, R14.P$2, U11.1.R/C
- removed net N$8: D11.DO, D12.DI
- removed net N$80: C22.P$1, U11.1.C
- removed net N$81: C23.P$2, R15.P$2, U11.2.R/C
- removed net N$82: C23.P$1, U11.2.C
- removed net TC0-ALRT1: U301.ALRT1@11
- removed net TC1-ALRT1: U302.ALRT1@11
- removed net WTIM0-CC0-ZERO-CROSS: U101.PE4
- new net D10-DO: D203.DO, D204.DI
- new net D11-DO: D204.DO, D205.DI
- new net D8-DI: D201.DI, TP201.S, U203.1.Y
- new net D8_DO: D201.DO, D202.DI
- new net D9-DO: D202.DO, D203.DI
- new net DVDD: C107.P$1, L101.P$1, U101.DVDD
- new net N$84: D206.3, J201.D+, JP202.2
- new net N$85: D206.2, J201.D-, JP201.2
- new net PA0: TP1.S, U101.PA0
- new net PA10: TP4.S, U101.PA10
- new net PA11: TP5.S, U101.PA11
- new net PA12: TP6.S, U101.PA12
- new net PA13: TP7.S, U101.PA13
- new net PA14: TP8.S, U101.PA14
- new net PA15: TP9.S, U101.PA15
- new net PA5: TP2.S, U101.PA5
- new net PA9: TP3.S, U101.PA9
- new net PB1: TP21.S, U101.PB1
- new net PB10: TP17.S, U101.PB10
- new net PB11: TP16.S, U101.PB11
- new net PB12: TP15.S, U101.PB12
- new net PB2: TP20.S, U101.PB2
- new net PB4: TP19.S, U101.PB4
- new net PB9: TP18.S, U101.PB9
- new net PC11: TP10.S, U101.PC11
- new net PE14: TP11.S, U101.PE14
- new net PE15: TP12.S, U101.PE15
- new net PF5: TP14.S, U101.PF5
- new net PF9: TP13.S, U101.PF9
- new net TFT-LEDK: Q201.C03, R204.P$1, R205.P$1
- new net TFT-LEDK1: R204.P$2, U204.LEDK@0
- new net TFT-LEDK2: R205.P$2, U204.LEDK@1
- new net U11.1-C: C201.P$1, U202.1.C
- new net U11.1-RC: C201.P$2, R201.P$2, U202.1.R/C
- new net U11.2-C: C202.P$1, U202.2.C
- new net U11.2-RC: C202.P$2, R202.P$2, U202.2.R/C
- new net U4-ALRT1: TP22.S, U301.ALRT1@11
- new net U7-ALRT1: TP26.S, U302.ALRT1@11
- new net VREGSW: L101.P$2, U101.VREGSW
- net !LED-CS: now also U202.1.!A, U202.2.!A; no longer U11.1.!A, U11.2.!A
- net !TFT_RESET: now also U204.!RESET; no longer U5.!RESET
- net !TTFT-IRQ: now also U204.X-/!IRQ!; no longer U5.X-/!IRQ!
- net !TTFT-RST: now also U204.Y-/!RST!; no longer U5.Y-/!RST!
- net 2.8V: now also C205.P$1, C206.P$1, C207.P$1, C208.P$1, C209.P$1, M201.VCC@9, R206.P$2, R209.P$1, R210.P$1, U201.PW.VCC, U204.!RD, U204.IM0, U204.IM1, U204.IM2, U204.VCI, U204.VDDI@0, U204.VDDI@1, U205.VDD@6, U205.VIO@5, U205.VREGIN@7; no longer C10.P$1, C11.P$1, C20.P$1, C26.P$1, C29.P$1, C6.P$1, C8.P$1, M1.VCC@9, R18.P$2, R34.P$1, R35.P$1, U$5.VIO@5, U5.!RD, U5.IM0, U5.IM1, U5.IM2, U5.VCI, U5.VDDI@0, U5.VDDI@1
- net 5V: now also C203.P$1, C204.P$1, D201.VDD, D202.VDD, D203.VDD, D204.VDD, D205.VDD, R201.P$1, R202.P$1, U202.1.!RD, U202.2.!RD, U202.PW.VCC, U203.PW.VCC, U204.LEDA; no longer C32.P$1, C35.P$1, D10.VDD, D11.VDD, D12.VDD, D8.VDD, D9.VDD, R14.P$1, R15.P$1, U11.1.!RD, U11.2.!RD, U11.PW.VCC, U13.PW.VCC, U5.LEDA
- net BLE-!RST: now also M201.!RST!@11; no longer M1.!RST!@11
- net BLE-KEY: now also M201.PIO0@16; no longer M1.PIO0@16
- net GND: now also C203.P$2, C204.P$2, C205.P$2, C206.P$2, C207.P$2, C208.P$2, C209.P$2, D201.VSS, D202.VSS, D203.VSS, D204.VSS, D205.VSS, D206.1, D208.CA, J201.CASE, J201.GND, M201.GND@12, Q201.EM2, R208.P$1, U201.PW.GND, U202.PW.GND, U203.PW.GND, U204.DB0, U204.DB1, U204.DB10, U204.DB11, U204.DB12, U204.DB13, U204.DB14, U204.DB15, U204.DB16, U204.DB17, U204.DB2, U204.DB3, U204.DB4, U204.DB5, U204.DB6, U204.DB7, U204.DB8, U204.DB9, U204.DE, U204.DOTCLK, U204.GND@0, U204.GND@1, U204.GND@2, U204.GND@3, U204.HSYNC, U204.TE, U204.VSYNC, U205.GND@2, U205.GND@PAD; no longer C10.P$2, C11.P$2, C20.P$2, C26.P$2, C27.P$2, C28.P$2, C29.P$2, C32.P$2, C35.P$2, C6.P$2, C8.P$2, D10.VSS, D11.VSS, D12.VSS, D4.1, D5.CA, D8.VSS, D9.VSS, J8.CASE, J8.GND, M1.GND@12, Q3.EM2, R38.P$1, U$5.GND@2, U$5.GND@PAD, U11.PW.GND, U12.PW.GND, U13.PW.GND, U5.DB0, U5.DB1, U5.DB10, U5.DB11, U5.DB12, U5.DB13, U5.DB14, U5.DB15, U5.DB16, U5.DB17, U5.DB2, U5.DB3, U5.DB4, U5.DB5, U5.DB6, U5.DB7, U5.DB8, U5.DB9, U5.DE, U5.DOTCLK, U5.GND@0, U5.GND@1, U5.GND@2, U5.GND@3, U5.HSYNC, U5.TE, U5.VSYNC
- net I2C1-SCL-TTFT: now also U204.X+/SCL; no longer U5.X+/SCL
- net I2C1-SDA-TTFT: now also U204.Y+/SDA; no longer U5.Y+/SDA
- net N$13: now also D207.CA, U205.GPIO1-RXT@13; no longer D3.CA, U$5.GPIO1-RXT@13
- net N$15: now also D209.CA, U205.GPIO0-TXT@14; no longer D2.CA, U$5.GPIO0-TXT@14
- net N$16: now also D209.AN, R210.P$2; no longer D2.AN, R34.P$2
- net N$19: now also D207.AN, R209.P$2; no longer D3.AN, R35.P$2
- net N$25: now also Q201.BA1, R203.P$2; no longer Q3.BA1, R24.P$2
- net N$35: now also D208.AN, R211.P$2; no longer D5.AN, R48.P$2
- net N$36: now also M201.PIO1@15, R211.P$1; no longer M1.PIO1@15, R48.P$1
- net N$51: now also D301.AN; no longer D7.AN
- net N$69: now also U202.2.Q, U203.1.B; no longer U11.2.Q, U13.1.B
- net N$7: now also D301.CA; no longer D7.CA
- net N$77: now also U202.1.Q, U203.1.A; no longer U11.1.Q, U13.1.A
- net N$78: now also U201.1.Y, U202.1.B; no longer U11.1.B, U12.1.Y
- net PRS-CH11-SSR-OUT: now also TP301.S
- net TFT-DC: now also U204.D/!C!; no longer U5.D/!C!
- net TIM1-CC0-TFT-BL: now also R203.P$1; no longer R24.P$1
- net U0RX-USB-TX: now also U205.TXD@21; no longer U$5.TXD@21
- net U0TX-USB-RX: now also U205.RXD@20; no longer U$5.RXD@20
- net U1RX-BLE-TX: now also M201.TX@2; no longer M1.TX@2
- net U1TX-BLE-RX: now also M201.RX@4; no longer M1.RX@4
- net UART_VBUS: now also R207.P$1, R208.P$2, U205.VBUS@8; no longer R37.P$1, R38.P$2, U$5.VBUS@8
- net US0-LED-MOSI: now also U201.1.A; no longer U12.1.A
- net US0-LED-SCK: now also U201.1.B, U202.2.B; no longer U11.2.B, U12.1.B
- net US1-CLK-TFT: now also U204.!WR!/SCL; no longer U5.!WR!/SCL
- net US1-CS-TFT: now also R206.P$1, U204.!CS; no longer R18.P$1, U5.!CS
- net US1-MISO-TFT: now also U204.SDO; no longer U5.SDO
- net US1-MOSI-TFT: now also U204.SDA; no longer U5.SDA
- net USB-D+: now also JP202.1; no longer D4.3, J8.VBUS, JP1.1, JP1.2
- net USB-D-: no longer D4.2, J8.D+, JP201.2
- net USB-ID: now also J201.ID; no longer J8._ID
- net USB-RST: now also U205.RSTB@9; no longer U$5.RSTB@9
- net USB-SUS: now also U205.SUSPEND@17; no longer U$5.SUSPEND@17
- net USB-UART-D+: now also JP202.3, U205.D+@3; no longer JP1.3, U$5.D+@3
- net USB-UART-D-: now also U205.D-@4; no longer U$5.D-@4
- net V_USB: now also D206.4, J201.VBUS, R207.P$2, TP202.S; no longer C27.P$1, D4.4, J8.D-, R37.P$2, U$5.VREGIN@7
- net WTIM1-CC1-ZERO-CROSS: now also TP302.S, U101.PE4
Other:
- note removed: "verify"
