File: pcb/hv0c.brd (EAGLE design)
At the start: 100 x 100 mm, 169 parts, among them J101 MICROSD, J102 SH-6, J201 USB-SHIELD, J301 PCC-SMP, J302 3X1_2.54, J303 3X1_2.54, J304 PCC-SMP, J305 2EDG-2P, J306 4P-PC-FAN, J307 2X1_2.54, J308 4P-PC-FAN, J401 2EDG-2P, M201 HM-11, Q201 BC817-40, Q202 BC817-40, Q301 BC817-40, Q302 BC817-40, Q303 BC817-40, Q304 MOC3051, Q305 BC817-40, Q306 BC817-40, Q307 BC817-40, Q308 BC817-40, U101 EFM32GG11B8XX_Q100, U102 SST26VF064B, U201 74LVC1G08, U202 74HC123, U203 74LVC1G32, U204 ER-TFT035-6BOT, U205 CP2102N, U301 MCP9600, U302 MCP9600, U303 H11AA1, U401 MIC4682, Y101 8MHz, Y102 32.768KHz

Commit message: sync
Parts:
- moved TP22 0.53 mm to (71.5, 11.1)
- moved C103 0.51 mm to (48.0, 74.5)
- moved TP17 0.41 mm to (60.6, 64.5)
- moved TP15 0.39 mm to (62.0, 64.5)
- moved TP8 0.28 mm to (59.1, 64.5)
- moved TP7 0.26 mm to (57.7, 61.8)
- moved TP16 0.17 mm to (59.3, 61.8)
- moved C101 0.15 mm to (51.5, 82.0)
- moved TP6 0.11 mm to (57.7, 64.5)
- moved TP18 0.05 mm to (61.3, 62.8)
Routing:
- net U4-ALRT1: track 3.26 -> 2.73 mm
- net GND: vias 425 -> 448
Other:
- outline, holes or cut-outs redrawn
- board text added: "Revision: hv0c Date: 05-19"
- board text removed: "Revision: hv0a Date: 05-19"
